File: CPU.kicad_sch (KiCad schematic)
At the start: 0 parts

Commit message: progress on switch sheet
Parts:
- added U801: MSP430F5507IRGZ, Package_DFN_QFN:Texas_RGZ0048A_VQFN-48-1EP_7x7mm_P0.5mm_EP5.15x5.15mm, symbol MCU_Texas_MSP430:MSP430F5507IRGZ
Changed lines of the file:
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@@
-		)
-	)
-	(text_box "CPU"
-		(exclude_from_sim no)
-		(at 108.204 94.996 0)
-		(size 44.45 85.09)
-		(margins 0.9525 0.9525 0.9525 0.9525)
-		(stroke
-			(width 0)
-			(type solid)
-		)
-		(fill
-			(type none)
-		)
-		(effects
-			(font
-				(size 1.27 1.27)
-			)
 		)
 	)
@@
 		)
 	)
+	(symbol
+		(lib_id "MCU_Texas_MSP430:MSP430F5507IRGZ")
+		(at 100.33 148.59 0)
+		(unit 1)
+		(exclude_from_sim no)
+		(in_bom yes)
+		(on_board yes)
+		(dnp no)
+		(fields_autoplaced yes)
+		(property "Reference" "U801"
+			(at 110.0933 179.07 0)
+			(effects
+				(font
+					(size 1.27 1.27)
+				)
+				(justify left)
+			)
+		)
+		(property "Value" "MSP430F5507IRGZ"
+			(at 110.0933 181.61 0)
+			(effects
+				(font
+					(size 1.27 1.27)
+				)
+				(justify left)
+			)
+		)
+		(property "Footprint" "Package_DFN_QFN:Texas_RGZ0048A_VQFN-48-1EP_7x7mm_P0.5mm_EP5.15x5.15mm"
+			(at 80.01 177.8 0)
+			(effects
+				(font
+					(size 1.27 1.27)
+					(italic yes)
+				)
+				(hide yes)
+			)
+		)
+		(property "Datasheet" "http://www.ti.com/lit/ds/symlink/msp430f5507.pdf"
+			(at 102.87 148.59 0)
+			(effects
+				(font
+					(size 1.27 1.27)
+				)
+				(hide yes)
+			)
+		)
+		(property "Description" "32kB Flash, 4kB + 2kB RAM, QFN-48"
+			(at 100.33 148.59 0)
+			(effects
+				(font
+					(size 1.27 1.27)
+				)
+				(hide yes)
+			)
+		)
+		(pin "36"
+		)
+		(pin "8"
+		)
+		(pin "29"
+		)
+		(pin "33"
+		)
+		(pin "46"
+		)
+		(pin "10"
+		)
+		(pin "43"
+		)
+		(pin "37"
+		)
+		(pin "45"
+		)
+		(pin "48"
+		)
+		(pin "47"
+		)
+		(pin "42"
+		)
+		(pin "23"
+		)
+		(pin "9"
+		)
+		(pin "26"
+		)
+		(pin "2"
+		)
+		(pin "12"
+		)
+		(pin "7"
+		)
+		(pin "20"
+		)
+		(pin "21"
+		)
+		(pin "5"
+		)
+		(pin "14"
+		)
+		(pin "22"
+		)
+		(pin "30"
+		)
+		(pin "32"
+		)
+		(pin "34"
+		)
+		(pin "17"
+		)
+		(pin "25"
+		)
+		(pin "28"
+		)
+		(pin "11"
+		)
+		(pin "27"
+		)
+		(pin "1"
+		)
+		(pin "41"
+		)
+		(pin "40"
+		)
+		(pin "24"
+		)
+		(pin "4"
+		)
+		(pin "3"
+		)
+		(pin "15"
+		)
+		(pin "39"
+		)
+		(pin "16"
+		)
+		(pin "6"
+		)
+		(pin "18"
+		)
+		(pin "44"
+		)
+		(pin "19"
+		)
+		(pin "38"
+		)
+		(pin "31"
+		)
+		(pin "35"
+		)
+		(pin "13"
+		)
+		(instances
+			(project "EPS"
+				(path "/94201994-47b8-4213-8d1a-05da12b2a7b0/436fb79f-2d07-4207-b819-4d05a5fd951c"
+					(reference "U801")
+					(unit 1)
+				)
+			)
+		)
+	)
