File: Switch.kicad_sch (KiCad schematic)
At the start: 40 parts, among them U1 TMCS1101A2UQDT, U12 MAX11604EEE+, U23 TCA9548APWR, U34 MCP4532T-104E/MS, U45 MAX890LESA+, U501 INA226, U56 AP22653AW6-7, U67 AP22653AW6-7

Commit message: specified design
Parts:
- removed C12, C501: 1uF, Capacitor_SMD:C_0603_1608Metric_Pad1.08x0.95mm_HandSolder, symbol Device:C_Small
- removed Q501, Q502, Q503: ~, Package_TO_SOT_SMD:TO-252-2, symbol Transistor_FET:RS9N50D
- removed R1, R12, R2, R23, R3, R34, R47, R48, R503, R504, R505, R506, R507, R508, R69, R70: 0R, symbol Device:R_Small
- removed R501: 1mR, symbol Device:R_Small
- removed R502, R509, R510, R511, R512, R515: 10kR, symbol Device:R_Small
- removed R513, R514, R516: 10R, symbol Device:R_Small
- removed U12: MAX11604EEE+, Package_SO:QSOP-16_3.9x4.9mm_P0.635mm, symbol Analog_ADC:MAX11616
- removed U23: TCA9548APWR, Package_SO:TSSOP-24_4.4x7.8mm_P0.65mm, symbol Interface_Expansion:TCA9548APWR
- removed U34: MCP4532T-104E/MS, Package_SO:TSSOP-14_4.4x5mm_P0.65mm, symbol Potentiometer_Digital:MCP45HV31-ST
- removed U45: MAX890LESA+, Package_DFN_QFN:DFN-8-1EP_3x3mm_P0.65mm_EP1.55x2.4mm, symbol Power_Management:MAX8586
- removed U501: INA226, Package_SO:VSSOP-10_3x3mm_P0.5mm, symbol Sensor_Energy:INA226
- removed U56, U67: AP22653AW6-7, Package_TO_SOT_SMD:SOT-23-6, symbol Regulator_Linear:AP22615AWU
- renumbered C1 to C901, U1 to U901
Connections:
- net VIN: no longer U901.1 (IP+), U901.2 (IP+)
- new net Switch_element/VOUT1: U901.1 (IP+), U901.2 (IP+)
- no-connect marks 7 -> 1
Other:
- added sheet Switch_element (Switch_element.kicad_sch)
- note removed: "FET ORing outputs? protection"
- note removed: "Later Will be outside the sheet combining outputs of multiple switches"
- note removed: "Real part has pin 3 and 4 reversed"
- note removed: "Switch"
- note removed: "will be dual with 2 rheostats"
- moved on the sheet: C901, U901
