File: TEST_PCB.kicad_pcb (KiCad board)
At the start: 6 copper layers, 90 x 95.8 mm, 305 parts, among them J101 Conn_01x07_Socket, J102 Conn_01x02_Socket, J103 Conn_01x04_Socket, J104 Conn_01x04_Socket, J105 Conn_01x02_Socket, J106 Conn_01x04_Socket, J107 Conn_01x02_Socket, J108 Conn_01x02_Socket, J109 Conn_01x04_Socket, J110 Conn_01x02_Socket, J111 Conn_01x02_Socket, J116 Conn_01x04_Socket, J117 Conn_01x02_Socket, J1901 PT_1000, J301 PT_1000, Q1101 NMOS, Q1102 NMOS, Q1201 NMOS, Q1202 NMOS, Q1203 NMOS, Q1901 IRLML5103, Q2001 NMOS, Q2002 NMOS, Q201 NMOS, Q202 NMOS, Q203 NMOS, Q204 NMOS, Q301 IRLML5103, Q501 NMOS, Q502 NMOS, Q503 NMOS, Q601 NMOS, Q602 NMOS, Q701 NMOS, Q702 NMOS, Q901 NMOS, Q902 NMOS, U1101 LM74700, U1102 LM74700, U1201 TPS62933, U1202 TPS62933, U1203 LM74700, U1204 LM74700, U1401 AP22653AW6-7, U1402 AP22653AW6-7, U1501 TMCS1101A2UQDT, U1701 AP22653AW6-7, U1702 AP22653AW6-7, U1801 AP22653AW6-7, U1802 AP22653AW6-7, U1901 ADA4807-1, U2001 LM74700, U2002 LM74700, U201 BQ24650, U2101 AP22653AW6-7, U2102 AP22653AW6-7, U2201 AP22653AW6-7, U2202 AP22653AW6-7, U301 ADA4807-1, U401 TMCS1101A2UQDT, U501 TPS62933, U502 TPS62933, U503 LM74700, U504 LM74700, U601 LM74700, U602 LM74700, U701 LM74700, U702 LM74700, U901 BQ76920PW

Commit message: restructurization of the entire project improved
Parts:
- removed BT901, BT902, BT903, BT904: Battery_Cell, Outlines:BHC186501P-li-ion
- removed C1201, C1202, C501, C502: TBD, Capacitor_SMD:C_0603_1608Metric_Pad1.08x0.95mm_HandSolder
- removed C1203, C1204, C302, C305, C503, C504: 10n, Capacitor_SMD:C_0603_1608Metric_Pad1.08x0.95mm_HandSolder
- removed C1205, C1206, C1207, C1208, C1209, C1210, C1211, C1212, C1213, C1214, C505, C506, C507, C508, C509, C510, C511, C512, C513, C514, C701, C702, C705, C706, C907, C908, C909: 100n, Capacitor_SMD:C_0603_1608Metric_Pad1.08x0.95mm_HandSolder
- removed C1215, C1216, C1217, C1218, C1704, C301, C515, C516, C517, C518, C703, C704: 1u, Capacitor_SMD:C_0603_1608Metric_Pad1.08x0.95mm_HandSolder
- removed C303: 10u, Capacitor_SMD:C_0603_1608Metric_Pad1.08x0.95mm_HandSolder
- removed C304: 3.3n, Capacitor_SMD:C_0603_1608Metric_Pad1.08x0.95mm_HandSolder
- removed C901, C902, C903, C904, C905, C906: 1uF, Capacitor_SMD:C_0603_1608Metric_Pad1.08x0.95mm_HandSolder
- removed C910: 10uF, Capacitor_SMD:C_0603_1608Metric_Pad1.08x0.95mm_HandSolder
- removed J101: Conn_01x07_Socket, Connector_PinSocket_2.54mm:PinSocket_1x07_P2.54mm_Vertical
- removed J106: Conn_01x04_Socket, Connector_PinSocket_2.54mm:PinSocket_1x02_P2.54mm_Vertical
- removed J108: Conn_01x02_Socket, Connector_PinSocket_2.54mm:PinSocket_1x02_P2.54mm_Vertical
- removed J1901, J301: PT_1000, Connector_PinSocket_1.00mm:PinSocket_1x02_P1.00mm_Vertical
- removed L1201, L1202: SELECT, Inductor_SMD:L_Taiyo-Yuden_NR-10050_9.8x10.0mm_HandSoldering
- removed L501, L502: SELECT, Inductor_SMD:L_6.3x6.3_H3
- removed Q1101, Q1102, Q1202, Q1203, Q502, Q503, Q701, Q702, Q901, Q902: NMOS, Outlines:NVTFS5116PLTWG
- removed Q1201, Q501: NMOS, Package_TO_SOT_SMD:SOT-23
- removed Q204: NMOS, Package_TO_SOT_SMD:SOT-23-3
- removed Q301: IRLML5103, Package_TO_SOT_SMD:SOT-23
- removed R101, R102, R106, R107, R1204, R1205, R504, R505: 0, Resistor_SMD:R_0603_1608Metric_Pad0.98x0.95mm_HandSolder
- removed R103, R1202, R1301, R1302, R1402, R1701, R1702, R215, R216, R301, R502: 100k, Resistor_SMD:R_0603_1608Metric_Pad0.98x0.95mm_HandSolder
- removed R104, R903, R904, R905, R906, R909, R910: 100, Resistor_SMD:R_0603_1608Metric_Pad0.98x0.95mm_HandSolder
- removed R1201, R1203, R501, R503: 10, Resistor_SMD:R_0603_1608Metric_Pad0.98x0.95mm_HandSolder
- removed R1206, R1207, R1208, R1209, R1403, R1404, R1703, R1704, R506, R507, R508, R509: SELECT, Resistor_SMD:R_0603_1608Metric_Pad0.98x0.95mm_HandSolder
- removed R1908, R308: 2k49, Resistor_SMD:R_0603_1608Metric
- removed R203: 500k, Resistor_SMD:R_0603_1608Metric_Pad0.98x0.95mm_HandSolder
- removed R217: 1k, Resistor_SMD:R_0603_1608Metric_Pad0.98x0.95mm_HandSolder
- removed R302: 10K, Resistor_SMD:R_0603_1608Metric
- removed R303: 39k, Resistor_SMD:R_0603_1608Metric
- removed R304: 22R, Resistor_SMD:R_0603_1608Metric
- removed R305: 100R, Resistor_SMD:R_0603_1608Metric
- removed R306: 1k, Resistor_SMD:R_0603_1608Metric
- removed R307: 150R, Resistor_SMD:R_0603_1608Metric
- removed R907: 20m, Resistor_SMD:R_0603_1608Metric_Pad0.98x0.95mm_HandSolder
- removed R908, R912, R913, R914, R915: 0R, Resistor_SMD:R_0603_1608Metric_Pad0.98x0.95mm_HandSolder
- removed R911, R916: 1M, Resistor_SMD:R_0603_1608Metric_Pad0.98x0.95mm_HandSolder
- removed TP101, TP102, TP901, TP902: ~, TestPoint:TestPoint_Pad_1.0x1.0mm
- removed U1101, U1102, U1203, U1204, U503, U504, U701, U702: LM74700, Package_TO_SOT_SMD:SOT-23-6
- removed U1201, U1202, U501, U502: TPS62933, Package_TO_SOT_SMD:SOT-583-8
- removed U1702, U1801, U1802, U2101, U2102, U2201, U2202: AP22653AW6-7, Package_TO_SOT_SMD:SOT-23-6
- removed U301: ADA4807-1, Package_TO_SOT_SMD:SOT-363_SC-70-6
- removed U901: BQ76920PW, Package_SO:TSSOP-20_4.4x6.5mm_P0.65mm
- added BT1001: Battery_Cell, Connector_PinSocket_2.54mm:PinSocket_1x02_P2.54mm_Vertical, F.Cu at (194.5, 122.9)
- added BT1002: Battery_Cell, Connector_PinSocket_2.54mm:PinSocket_1x02_P2.54mm_Vertical, F.Cu at (194.5, 116.8)
- added BT1003: Battery_Cell, Connector_PinSocket_2.54mm:PinSocket_1x02_P2.54mm_Vertical, F.Cu at (194.5, 110.7)
- added BT1004: Battery_Cell, Connector_PinSocket_2.54mm:PinSocket_1x02_P2.54mm_Vertical, F.Cu at (194.5, 104.6)
- added C1001: 1uF, Capacitor_SMD:C_0603_1608Metric_Pad1.08x0.95mm_HandSolder, F.Cu at (189.4, 118.1)
- added C1002: 1uF, Capacitor_SMD:C_0603_1608Metric_Pad1.08x0.95mm_HandSolder, F.Cu at (189.4, 114.2)
- added C1003: 1uF, Capacitor_SMD:C_0603_1608Metric_Pad1.08x0.95mm_HandSolder, F.Cu at (189.4, 110.6)
- added C1004: 1uF, Capacitor_SMD:C_0603_1608Metric_Pad1.08x0.95mm_HandSolder, F.Cu at (189.4, 106.9)
- added C1005: 1uF, Capacitor_SMD:C_0603_1608Metric_Pad1.08x0.95mm_HandSolder, F.Cu at (173.5, 111.2)
- added C1006: 1uF, Capacitor_SMD:C_0603_1608Metric_Pad1.08x0.95mm_HandSolder, F.Cu at (173.8, 115.1)
- added C1007: 100n, Capacitor_SMD:C_0603_1608Metric_Pad1.08x0.95mm_HandSolder, F.Cu at (187.0, 105.6)
- added C1008: 100n, Capacitor_SMD:C_0603_1608Metric_Pad1.08x0.95mm_HandSolder, F.Cu at (181.9, 105.6)
- added C1009: 100n, Capacitor_SMD:C_0603_1608Metric_Pad1.08x0.95mm_HandSolder, F.Cu at (184.4, 106.5)
- added C101: 1u, Capacitor_SMD:C_0603_1608Metric_Pad1.08x0.95mm_HandSolder, F.Cu at (242.4, 58.4)
- added C1010: 10uF, Capacitor_SMD:C_0603_1608Metric_Pad1.08x0.95mm_HandSolder, F.Cu at (180.6, 116.1)
- added C102: 100n, Capacitor_SMD:C_0603_1608Metric_Pad1.08x0.95mm_HandSolder, F.Cu at (242.4, 60.2)
- added C103: 100n, Capacitor_SMD:C_0603_1608Metric_Pad1.08x0.95mm_HandSolder, F.Cu at (242.9, 67.6)
- added C104: 1u, Capacitor_SMD:C_0603_1608Metric_Pad1.08x0.95mm_HandSolder, F.Cu at (242.9, 69.4)
- added C105: 100n, Capacitor_SMD:C_0603_1608Metric_Pad1.08x0.95mm_HandSolder, F.Cu at (242.9, 65.9)
- added C1107: 1u, Capacitor_SMD:C_0603_1608Metric_Pad1.08x0.95mm_HandSolder, F.Cu at (211.0, 103.0)
- added C1108: 1u, Capacitor_SMD:C_0603_1608Metric_Pad1.08x0.95mm_HandSolder, F.Cu at (211.2, 115.8)
- added C1405: 100n, Capacitor_SMD:C_0603_1608Metric_Pad1.08x0.95mm_HandSolder, F.Cu at (185.2, 77.6)
- added C1406: 100n, Capacitor_SMD:C_0603_1608Metric_Pad1.08x0.95mm_HandSolder, F.Cu at (184.8, 89.2)
- added C1504: 10u, Capacitor_SMD:C_0603_1608Metric_Pad1.08x0.95mm_HandSolder, F.Cu at (177.7, 65.6)
- added C1505: 100n, Capacitor_SMD:C_0603_1608Metric_Pad1.08x0.95mm_HandSolder, F.Cu at (176.7, 53.9)
- added C1506: 100n, Capacitor_SMD:C_0603_1608Metric_Pad1.08x0.95mm_HandSolder, F.Cu at (175.9, 65.6)
- added C1507: 10n, Capacitor_SMD:C_0603_1608Metric_Pad1.08x0.95mm_HandSolder, F.Cu at (182.8, 50.4)
- added C1508: 10n, Capacitor_SMD:C_0603_1608Metric_Pad1.08x0.95mm_HandSolder, F.Cu at (184.9, 62.4)
- added C1509: 100n, Capacitor_SMD:C_0603_1608Metric_Pad1.08x0.95mm_HandSolder, F.Cu at (182.7, 54.0)
- added C1510: 100n, Capacitor_SMD:C_0603_1608Metric_Pad1.08x0.95mm_HandSolder, F.Cu at (184.9, 66.0)
- added C1511: 100n, Capacitor_SMD:C_0603_1608Metric_Pad1.08x0.95mm_HandSolder, F.Cu at (179.6, 55.1)
- added C1512: 100n, Capacitor_SMD:C_0603_1608Metric_Pad1.08x0.95mm_HandSolder, F.Cu at (182.1, 66.5)
- added C1513: 10u, Capacitor_SMD:C_0603_1608Metric_Pad1.08x0.95mm_HandSolder, F.Cu at (197.1, 50.6)
- added C1514: 10u, Capacitor_SMD:C_0603_1608Metric_Pad1.08x0.95mm_HandSolder, F.Cu at (198.5, 62.9)
- added C1515: 10u, Capacitor_SMD:C_0603_1608Metric_Pad1.08x0.95mm_HandSolder, F.Cu at (195.5, 54.2)
- added C1516: 10u, Capacitor_SMD:C_0603_1608Metric_Pad1.08x0.95mm_HandSolder, F.Cu at (198.4, 66.4)
- added C1517: 10u, Capacitor_SMD:C_0603_1608Metric_Pad1.08x0.95mm_HandSolder, F.Cu at (197.1, 54.2)
- added C1518: 10u, Capacitor_SMD:C_0603_1608Metric_Pad1.08x0.95mm_HandSolder, F.Cu at (196.8, 66.4)
- added C1519: 10u, Capacitor_SMD:C_0603_1608Metric_Pad1.08x0.95mm_HandSolder, F.Cu at (195.4, 50.6)
- added C1520: 10u, Capacitor_SMD:C_0603_1608Metric_Pad1.08x0.95mm_HandSolder, F.Cu at (196.8, 62.9)
- added C1521: 1u, Capacitor_SMD:C_0603_1608Metric_Pad1.08x0.95mm_HandSolder, F.Cu at (200.7, 49.7)
- added C1522: 1u, Capacitor_SMD:C_0603_1608Metric_Pad1.08x0.95mm_HandSolder, F.Cu at (202.2, 62.1)
- added C1523: 1u, Capacitor_SMD:C_0603_1608Metric_Pad1.08x0.95mm_HandSolder, F.Cu at (200.7, 55.2)
- added C1524: 1u, Capacitor_SMD:C_0603_1608Metric_Pad1.08x0.95mm_HandSolder, F.Cu at (202.2, 67.5)
- added C1805: 1u, Capacitor_SMD:C_0603_1608Metric_Pad1.08x0.95mm_HandSolder, F.Cu at (130.5, 107.8)
- added C1806: 1u, Capacitor_SMD:C_0603_1608Metric_Pad1.08x0.95mm_HandSolder, F.Cu at (130.1, 120.8)
- added C1807: 1u, Capacitor_SMD:C_0603_1608Metric_Pad1.08x0.95mm_HandSolder, F.Cu at (130.6, 104.1)
- added C1808: 1u, Capacitor_SMD:C_0603_1608Metric_Pad1.08x0.95mm_HandSolder, F.Cu at (130.1, 117.2)
- added C209: 1u, Capacitor_SMD:C_0603_1608Metric_Pad1.08x0.95mm_HandSolder, F.Cu at (94.5, 119.6)
- added C2105: 1u, Capacitor_SMD:C_0603_1608Metric_Pad1.08x0.95mm_HandSolder, F.Cu at (237.3, 104.7)
- added C2106: 1u, Capacitor_SMD:C_0603_1608Metric_Pad1.08x0.95mm_HandSolder, F.Cu at (237.2, 125.0)
- added C2107: 1u, Capacitor_SMD:C_0603_1608Metric_Pad1.08x0.95mm_HandSolder, F.Cu at (230.7, 97.9)
- added C2108: 1u, Capacitor_SMD:C_0603_1608Metric_Pad1.08x0.95mm_HandSolder, F.Cu at (230.2, 117.6)
- added C2205: 1u, Capacitor_SMD:C_0603_1608Metric_Pad1.08x0.95mm_HandSolder, F.Cu at (179.6, 76.3)
- added C2206: 1u, Capacitor_SMD:C_0603_1608Metric_Pad1.08x0.95mm_HandSolder, F.Cu at (179.4, 87.9)
- added C2207: 1u, Capacitor_SMD:C_0603_1608Metric_Pad1.08x0.95mm_HandSolder, F.Cu at (179.6, 72.7)
- added C2208: 1u, Capacitor_SMD:C_0603_1608Metric_Pad1.08x0.95mm_HandSolder, F.Cu at (179.4, 84.4)
- added C2301: 1u, Capacitor_SMD:C_0603_1608Metric_Pad1.08x0.95mm_HandSolder, F.Cu at (222.7, 61.5)
- added C2302: 1u, Capacitor_SMD:C_0603_1608Metric_Pad1.08x0.95mm_HandSolder, F.Cu at (223.0, 50.4)
- added C2303: 1u, Capacitor_SMD:C_0603_1608Metric_Pad1.08x0.95mm_HandSolder, F.Cu at (224.2, 68.7)
- added C2304: 1u, Capacitor_SMD:C_0603_1608Metric_Pad1.08x0.95mm_HandSolder, F.Cu at (224.5, 57.7)
- added C2305: 1u, Capacitor_SMD:C_0603_1608Metric_Pad1.08x0.95mm_HandSolder, F.Cu at (232.5, 64.0)
- added C2306: 1u, Capacitor_SMD:C_0603_1608Metric_Pad1.08x0.95mm_HandSolder, F.Cu at (232.5, 54.6)
- added C2307: 1u, Capacitor_SMD:C_0603_1608Metric_Pad1.08x0.95mm_HandSolder, F.Cu at (234.2, 64.0)
- added C2308: 1u, Capacitor_SMD:C_0603_1608Metric_Pad1.08x0.95mm_HandSolder, F.Cu at (232.5, 51.0)
- added C801: 100n, Capacitor_SMD:C_0603_1608Metric_Pad1.08x0.95mm_HandSolder, F.Cu at (214.5, 107.3)
- added C802: 100n, Capacitor_SMD:C_0603_1608Metric_Pad1.08x0.95mm_HandSolder, F.Cu at (216.3, 115.0)
- added C803: 1u, Capacitor_SMD:C_0603_1608Metric_Pad1.08x0.95mm_HandSolder, F.Cu at (218.1, 107.3)
- added H105: MountingHole, MountingHole:MountingHole_3.2mm_M3_Pad_TopBottom, F.Cu at (151.7, 133.8)
- added H106: MountingHole, MountingHole:MountingHole_3.2mm_M3_Pad_TopBottom, F.Cu at (71.7, 133.8)
- added H107: MountingHole, MountingHole:MountingHole_3.2mm_M3_Pad_TopBottom, F.Cu at (75.5, 48.1)
- added H108: MountingHole, MountingHole:MountingHole_3.2mm_M3_Pad_TopBottom, F.Cu at (149.2, 48.1)
- added IC1101: TPS259802ONRGER, Outlines:TPS259802ONRGER, F.Cu at (206.5, 104.5)
- added IC1102: TPS259802ONRGER, Outlines:TPS259802ONRGER, F.Cu at (206.6, 117.5)
- added IC1801: TPS259802ONRGER, Outlines:TPS259802ONRGER, F.Cu at (126.1, 105.5)
- added IC1802: TPS259802ONRGER, Outlines:TPS259802ONRGER, F.Cu at (125.8, 118.2)
- added IC2101: TPS259802ONRGER, Outlines:TPS259802ONRGER, F.Cu at (233.0, 102.3)
- added IC2102: TPS259802ONRGER, Outlines:TPS259802ONRGER, F.Cu at (232.5, 122.2)
- added IC2201: TPS259802ONRGER, Outlines:TPS259802ONRGER, F.Cu at (175.1, 74.1)
- added IC2202: TPS259802ONRGER, Outlines:TPS259802ONRGER, F.Cu at (174.8, 86.1)
- added IC2301: TPS259802ONRGER, Outlines:TPS259802ONRGER, F.Cu at (227.8, 63.2)
- added IC2302: TPS259802ONRGER, Outlines:TPS259802ONRGER, F.Cu at (228.1, 52.4)
- added J1001: PT_1000, Connector_PinSocket_2.54mm:PinSocket_1x02_P2.54mm_Vertical, F.Cu at (187.6, 133.8)
- added J112: Conn_01x02_Socket, Connector_PinSocket_2.54mm:PinSocket_1x02_P2.54mm_Vertical, F.Cu at (166.4, 81.1)
- added J113: Conn_01x03_Pin, Connector_PinSocket_2.54mm:PinSocket_1x02_P2.54mm_Vertical, F.Cu at (222.0, 110.0)
- added J114: Conn_01x02_Pin, Connector_PinSocket_2.54mm:PinSocket_1x02_P2.54mm_Vertical, F.Cu at (189.0, 80.9)
- added J115: Conn_01x02_Socket, Connector_PinSocket_2.54mm:PinSocket_1x02_P2.54mm_Vertical, F.Cu at (181.2, 92.1)
- added J118: Conn_01x02_Socket, Connector_PinHeader_2.54mm:PinHeader_1x03_P2.54mm_Vertical, F.Cu at (223.7, 73.1)
- added J119: Conn_01x02_Socket, Connector_PinSocket_2.54mm:PinSocket_1x02_P2.54mm_Vertical, F.Cu at (219.7, 57.9)
- added J120: Conn_01x02_Pin, Connector_PinSocket_2.54mm:PinSocket_1x02_P2.54mm_Vertical, F.Cu at (237.2, 57.8)
- added J121: Conn_01x02_Socket, Connector_PinSocket_2.54mm:PinSocket_1x02_P2.54mm_Vertical, F.Cu at (235.6, 73.1)
- added J122: Conn_01x02_Pin, Connector_PinSocket_2.54mm:PinSocket_1x02_P2.54mm_Vertical, F.Cu at (239.9, 78.3)
- added J123: Conn_01x02_Socket, Connector_PinSocket_2.54mm:PinSocket_1x02_P2.54mm_Vertical, F.Cu at (226.0, 78.5)
- added J124: Conn_01x02_Socket, Connector_PinSocket_2.54mm:PinSocket_1x02_P2.54mm_Vertical, F.Cu at (243.6, 80.7)
- added J125: Conn_01x02_Pin, Connector_PinSocket_2.54mm:PinSocket_1x02_P2.54mm_Vertical, F.Cu at (136.1, 112.7)
- added J126: Conn_01x02_Socket, Connector_PinHeader_2.54mm:PinHeader_1x02_P2.54mm_Vertical, F.Cu at (195.5, 80.9)
- added J127: Conn_01x03_Pin, Connector_PinHeader_2.54mm:PinHeader_1x02_P2.54mm_Vertical, F.Cu at (143.1, 112.7)
- added J128: Conn_01x02_Pin, Connector_PinHeader_2.54mm:PinHeader_1x02_P2.54mm_Vertical, F.Cu at (209.1, 58.0)
- added J129: Conn_01x02_Socket, Connector_PinHeader_2.54mm:PinHeader_1x02_P2.54mm_Vertical, F.Cu at (237.3, 64.3)
- added J130: Conn_01x02_Socket, Connector_PinHeader_2.54mm:PinHeader_1x02_P2.54mm_Vertical, F.Cu at (147.1, 120.3)
- added J132: Conn_01x02_Pin, Connector_PinSocket_2.54mm:PinSocket_1x03_P2.54mm_Vertical, F.Cu at (92.2, 102.7)
- added J133: Conn_01x02_Socket, Connector_PinSocket_2.54mm:PinSocket_1x03_P2.54mm_Vertical, F.Cu at (92.2, 100.1)
- added J134: Conn_01x02_Socket, Connector_PinHeader_2.54mm:PinHeader_1x02_P2.54mm_Vertical, F.Cu at (212.1, 52.3)
- added J135: Conn_01x02_Socket, Connector_PinHeader_2.54mm:PinHeader_1x02_P2.54mm_Vertical, F.Cu at (240.7, 72.4)
- added J137: Conn_01x05_Socket, Connector_PinSocket_2.54mm:PinSocket_1x05_P2.54mm_Vertical, F.Cu at (76.0, 119.7)
- added J139: Conn_01x02_Socket, Connector_PinSocket_2.54mm:PinSocket_1x02_P2.54mm_Vertical, F.Cu at (168.2, 112.3)
- added J140: Conn_01x02_Socket, Connector_PinSocket_2.54mm:PinSocket_1x02_P2.54mm_Vertical, F.Cu at (217.5, 117.8)
- added J141: Conn_01x02_Socket, Connector_PinSocket_2.54mm:PinSocket_1x02_P2.54mm_Vertical, F.Cu at (223.0, 86.9)
- added J142: Conn_01x02_Socket, Connector_PinSocket_2.54mm:PinSocket_1x02_P2.54mm_Vertical, F.Cu at (147.2, 124.4)
- added J201: PT_1000, Connector_PinSocket_2.54mm:PinSocket_1x02_P2.54mm_Vertical, F.Cu at (101.3, 102.9)
- added L1501: SELECT, Inductor_SMD:L_Vishay_IHLP-2525, F.Cu at (189.5, 52.2)
- added L1502: SELECT, Inductor_SMD:L_Vishay_IHLP-2525, F.Cu at (190.0, 63.5)
- added PCB102: PCB Outline, Outlines:SPACEMANIC_V1c, F.Cu at (111.7, 91.0)
- added Q1001: NVTFWS4D9N04XMTAG, Outlines:NVTFS5116PLTWG, F.Cu at (178.3, 99.2)
- added Q1002: NVTFWS4D9N04XMTAG, Outlines:NVTFS5116PLTWG, F.Cu at (171.7, 99.3)
- added Q1401: NVTFWS4D9N04XMTAG, Outlines:NVTFS5116PLTWG, F.Cu at (191.1, 75.6)
- added Q1402: NVTFWS4D9N04XMTAG, Outlines:NVTFS5116PLTWG, F.Cu at (190.2, 87.4)
- added Q1501: IRLML5103, Package_TO_SOT_SMD:SOT-23, F.Cu at (168.0, 58.6)
- added Q1502: NVTFWS4D9N04XMTAG, Outlines:NVTFS5116PLTWG, F.Cu at (206.8, 51.3)
- added Q1503: NVTFWS4D9N04XMTAG, Outlines:NVTFS5116PLTWG, F.Cu at (207.9, 63.9)
- added R1001: 100k, Resistor_SMD:R_0603_1608Metric_Pad0.98x0.95mm_HandSolder, F.Cu at (187.7, 128.5)
- added R1002: 100k, Resistor_SMD:R_0603_1608Metric_Pad0.98x0.95mm_HandSolder, F.Cu at (191.3, 120.0)
- added R1003: 100, Resistor_SMD:R_0603_1608Metric_Pad0.98x0.95mm_HandSolder, F.Cu at (191.3, 116.3)
- added R1004: 100, Resistor_SMD:R_0603_1608Metric_Pad0.98x0.95mm_HandSolder, F.Cu at (191.3, 112.6)
- added R1005: 100, Resistor_SMD:R_0603_1608Metric_Pad0.98x0.95mm_HandSolder, F.Cu at (191.3, 108.8)
- added R1006: 100, Resistor_SMD:R_0603_1608Metric_Pad0.98x0.95mm_HandSolder, F.Cu at (191.3, 105.0)
- added R1007: 100, Resistor_SMD:R_0603_1608Metric_Pad0.98x0.95mm_HandSolder, F.Cu at (185.2, 103.7)
- added R1008: 20m, Resistor_SMD:R_1210_3225Metric_Pad1.30x2.65mm_HandSolder, F.Cu at (185.2, 98.3)
- added R1009: 100, Resistor_SMD:R_0603_1608Metric_Pad0.98x0.95mm_HandSolder, F.Cu at (176.9, 116.1)
- added R1010: 100, Resistor_SMD:R_0603_1608Metric_Pad0.98x0.95mm_HandSolder, F.Cu at (183.5, 103.7)
- added R1011: 1M, Resistor_SMD:R_0603_1608Metric_Pad0.98x0.95mm_HandSolder, F.Cu at (178.8, 106.8)
- added R1012: 0, Resistor_SMD:R_1210_3225Metric_Pad1.30x2.65mm_HandSolder, F.Cu at (178.2, 104.2)
- added R1013: 0, Resistor_SMD:R_1210_3225Metric_Pad1.30x2.65mm_HandSolder, F.Cu at (171.8, 104.2)
- added R1014: 1M, Resistor_SMD:R_0603_1608Metric_Pad0.98x0.95mm_HandSolder, F.Cu at (170.4, 107.0)
- added R109: 100k, Resistor_SMD:R_0603_1608Metric_Pad0.98x0.95mm_HandSolder, F.Cu at (166.3, 84.2)
- added R110: 100, Resistor_SMD:R_0603_1608Metric_Pad0.98x0.95mm_HandSolder, F.Cu at (166.3, 86.1)
- added R1101: 100k, Resistor_SMD:R_0603_1608Metric_Pad0.98x0.95mm_HandSolder, F.Cu at (201.0, 106.1)
- added R1102: 100k, Resistor_SMD:R_0603_1608Metric_Pad0.98x0.95mm_HandSolder, F.Cu at (201.3, 119.3)
- added R1103: 0, Resistor_SMD:R_0603_1608Metric_Pad0.98x0.95mm_HandSolder, F.Cu at (207.9, 110.1)
- added R1104: 0, Resistor_SMD:R_0603_1608Metric_Pad0.98x0.95mm_HandSolder, F.Cu at (207.8, 123.2)
- added R1105: 0, Resistor_SMD:R_0603_1608Metric_Pad0.98x0.95mm_HandSolder, F.Cu at (206.3, 110.1)
- added R1106: 0, Resistor_SMD:R_0603_1608Metric_Pad0.98x0.95mm_HandSolder, F.Cu at (206.2, 123.2)
- added R1107: SELECT, Resistor_SMD:R_0603_1608Metric_Pad0.98x0.95mm_HandSolder, F.Cu at (204.7, 110.1)
- added R1108: SELECT, Resistor_SMD:R_0603_1608Metric_Pad0.98x0.95mm_HandSolder, F.Cu at (204.6, 123.2)
- added R1109: 0, Resistor_SMD:R_0603_1608Metric_Pad0.98x0.95mm_HandSolder, F.Cu at (209.5, 110.1)
- added R1110: 0, Resistor_SMD:R_0603_1608Metric_Pad0.98x0.95mm_HandSolder, F.Cu at (209.4, 123.2)
- added R1501: 10, Resistor_SMD:R_0603_1608Metric_Pad0.98x0.95mm_HandSolder, F.Cu at (163.2, 58.6)
- added R1502: 100k, Resistor_SMD:R_0603_1608Metric_Pad0.98x0.95mm_HandSolder, F.Cu at (167.9, 55.6)
- added R1503: 10, Resistor_SMD:R_0603_1608Metric_Pad0.98x0.95mm_HandSolder, F.Cu at (165.0, 57.3)
- added R1504: 0, Resistor_SMD:R_0603_1608Metric_Pad0.98x0.95mm_HandSolder, F.Cu at (175.7, 51.3)
- added R1505: 0, Resistor_SMD:R_0603_1608Metric_Pad0.98x0.95mm_HandSolder, F.Cu at (178.5, 62.5)
- added R1506: SELECT, Resistor_SMD:R_0603_1608Metric_Pad0.98x0.95mm_HandSolder, F.Cu at (178.5, 48.9)
- added R1507: SELECT, Resistor_SMD:R_0603_1608Metric_Pad0.98x0.95mm_HandSolder, F.Cu at (180.4, 48.8)
- added R1508: SELECT, Resistor_SMD:R_0603_1608Metric_Pad0.98x0.95mm_HandSolder, F.Cu at (183.0, 60.7)
- added R1509: SELECT, Resistor_SMD:R_0603_1608Metric_Pad0.98x0.95mm_HandSolder, F.Cu at (181.2, 60.7)
- added R1601: 100k, Resistor_SMD:R_0603_1608Metric_Pad0.98x0.95mm_HandSolder, F.Cu at (222.7, 57.7)
- added R1602: 100k, Resistor_SMD:R_0603_1608Metric_Pad0.98x0.95mm_HandSolder, F.Cu at (222.5, 68.7)
- added R1805: 0, Resistor_SMD:R_0603_1608Metric_Pad0.98x0.95mm_HandSolder, F.Cu at (126.0, 111.5)
- added R1806: 0, Resistor_SMD:R_0603_1608Metric_Pad0.98x0.95mm_HandSolder, F.Cu at (125.1, 124.1)
- added R1807: SELECT, Resistor_SMD:R_0603_1608Metric_Pad0.98x0.95mm_HandSolder, F.Cu at (124.4, 111.5)
- added R1808: SELECT, Resistor_SMD:R_0603_1608Metric_Pad0.98x0.95mm_HandSolder, F.Cu at (123.5, 124.1)
- added R1809: 0, Resistor_SMD:R_0603_1608Metric_Pad0.98x0.95mm_HandSolder, F.Cu at (129.2, 111.5)
- added R1810: 0, Resistor_SMD:R_0603_1608Metric_Pad0.98x0.95mm_HandSolder, F.Cu at (128.3, 124.1)
- added R2001: 100k, Resistor_SMD:R_0603_1608Metric_Pad0.98x0.95mm_HandSolder, F.Cu at (225.0, 124.1)
- added R2105: 0, Resistor_SMD:R_0603_1608Metric_Pad0.98x0.95mm_HandSolder, F.Cu at (232.7, 108.2)
- added R2106: 0, Resistor_SMD:R_0603_1608Metric_Pad0.98x0.95mm_HandSolder, F.Cu at (232.1, 128.1)
- added R2107: SELECT, Resistor_SMD:R_0603_1608Metric_Pad0.98x0.95mm_HandSolder, F.Cu at (231.1, 108.2)
- added R2108: SELECT, Resistor_SMD:R_0603_1608Metric_Pad0.98x0.95mm_HandSolder, F.Cu at (230.5, 128.1)
- added R2109: 0, Resistor_SMD:R_0603_1608Metric_Pad0.98x0.95mm_HandSolder, F.Cu at (235.8, 108.2)
- added R2110: 0, Resistor_SMD:R_0603_1608Metric_Pad0.98x0.95mm_HandSolder, F.Cu at (235.3, 128.1)
- added R2205: 0, Resistor_SMD:R_0603_1608Metric_Pad0.98x0.95mm_HandSolder, F.Cu at (174.9, 79.9)
- added R2206: 0, Resistor_SMD:R_0603_1608Metric_Pad0.98x0.95mm_HandSolder, F.Cu at (175.0, 91.9)
- added R2207: SELECT, Resistor_SMD:R_0603_1608Metric_Pad0.98x0.95mm_HandSolder, F.Cu at (173.3, 79.9)
- added R2208: SELECT, Resistor_SMD:R_0603_1608Metric_Pad0.98x0.95mm_HandSolder, F.Cu at (173.4, 91.9)
- added R2209: 0, Resistor_SMD:R_0603_1608Metric_Pad0.98x0.95mm_HandSolder, F.Cu at (178.1, 79.9)
- added R2210: 0, Resistor_SMD:R_0603_1608Metric_Pad0.98x0.95mm_HandSolder, F.Cu at (178.2, 91.9)
- added R2301: 100k, Resistor_SMD:R_0603_1608Metric_Pad0.98x0.95mm_HandSolder, F.Cu at (222.7, 65.1)
- added R2302: 100k, Resistor_SMD:R_0603_1608Metric_Pad0.98x0.95mm_HandSolder, F.Cu at (223.0, 53.9)
- added R2303: 0, Resistor_SMD:R_0603_1608Metric_Pad0.98x0.95mm_HandSolder, F.Cu at (229.3, 68.7)
- added R2304: 0, Resistor_SMD:R_0603_1608Metric_Pad0.98x0.95mm_HandSolder, F.Cu at (229.3, 57.7)
- added R2305: 0, Resistor_SMD:R_0603_1608Metric_Pad0.98x0.95mm_HandSolder, F.Cu at (227.6, 68.7)
- added R2306: 0, Resistor_SMD:R_0603_1608Metric_Pad0.98x0.95mm_HandSolder, F.Cu at (227.7, 57.7)
- added R2307: SELECT, Resistor_SMD:R_0603_1608Metric_Pad0.98x0.95mm_HandSolder, F.Cu at (225.9, 68.7)
- added R2308: SELECT, Resistor_SMD:R_0603_1608Metric_Pad0.98x0.95mm_HandSolder, F.Cu at (226.1, 57.7)
- added R2309: 0, Resistor_SMD:R_0603_1608Metric_Pad0.98x0.95mm_HandSolder, F.Cu at (231.0, 68.7)
- added R2310: 0, Resistor_SMD:R_0603_1608Metric_Pad0.98x0.95mm_HandSolder, F.Cu at (230.9, 57.7)
- added R601: 100k, Resistor_SMD:R_0603_1608Metric_Pad0.98x0.95mm_HandSolder, F.Cu at (120.3, 124.1)
- added TP1001: ~, TestPoint:TestPoint_Pad_1.0x1.0mm, F.Cu at (173.6, 107.3)
- added TP1002: ~, TestPoint:TestPoint_Pad_1.0x1.0mm, F.Cu at (169.9, 108.9)
- added U1001: BQ76920PW, Package_SO:TSSOP-20_4.4x6.5mm_P0.65mm, F.Cu at (179.1, 111.4)
- added U101: LP38690SDX-3.3/NOPB, Package_SON:WSON-6-1EP_3x3mm_P0.95mm, F.Cu at (242.6, 63.0)
- added U1502: TPS62933, Package_TO_SOT_SMD:SOT-583-8, F.Cu at (182.1, 64.0)
- added U1503: LM74700, Package_TO_SOT_SMD:SOT-23-6, F.Cu at (200.7, 52.4)
- added U1504: LM74700, Package_TO_SOT_SMD:SOT-23-6, F.Cu at (202.2, 64.8)
- added U801: LM74700, Package_SO:SOIC-8_3.9x4.9mm_P1.27mm, F.Cu at (216.3, 111.1)
- C1101, C1102, C1105, C1106: value 100n -> 1u
- C1401, C1402, C401, C402: value 1u -> 100n
- C1501, C1502: value 1u -> TBD
- C1503: value 1u -> 10u
- H101, H102, H103, H104: footprint MountingHole:MountingHole_3.2mm_M3_Pad_Via -> MountingHole:MountingHole_3.2mm_M3_Pad_TopBottom
- J102: value Conn_01x02_Socket -> Conn_01x05_Socket; footprint Connector_PinSocket_2.54mm:PinSocket_1x04_P2.54mm_Vertical -> Connector_PinSocket_2.54mm:PinSocket_1x05_P2.54mm_Vertical
- J103, J109: value Conn_01x04_Socket -> Conn_01x02_Socket; footprint Connector_PinSocket_2.54mm:PinSocket_1x04_P2.54mm_Vertical -> Connector_PinSocket_2.54mm:PinSocket_1x02_P2.54mm_Vertical
- J104: footprint Connector_PinSocket_2.54mm:PinSocket_1x02_P2.54mm_Vertical -> Connector_PinSocket_2.54mm:PinSocket_1x04_P2.54mm_Vertical
- J105: value Conn_01x02_Socket -> Conn_01x03_Pin; footprint Connector_PinSocket_2.54mm:PinSocket_1x04_P2.54mm_Vertical -> Connector_PinHeader_2.54mm:PinHeader_1x03_P2.54mm_Vertical
- J107: value Conn_01x02_Socket -> Conn_01x03_Socket
- J110: value Conn_01x02_Socket -> Conn_01x03_Socket; footprint Connector_PinSocket_2.54mm:PinSocket_1x02_P2.54mm_Vertical -> Connector_PinHeader_2.54mm:PinHeader_1x03_P2.54mm_Vertical
- J111: value Conn_01x02_Socket -> Conn_01x02_Pin
- J116: value Conn_01x04_Socket -> Conn_01x02_Socket; footprint Connector_PinSocket_2.54mm:PinSocket_1x02_P2.54mm_Vertical -> Connector_PinHeader_2.54mm:PinHeader_1x02_P2.54mm_Vertical
- Q2001, Q2002, Q202, Q203, Q601, Q602: value NMOS -> NVTFWS4D9N04XMTAG
- Q201: value NMOS -> IRLML5103
- R105, RSR201: footprint Resistor_SMD:R_0603_1608Metric_Pad0.98x0.95mm_HandSolder -> Resistor_SMD:R_1210_3225Metric_Pad1.30x2.65mm_HandSolder
- R1803, R1804, R2103, R2104, R2203, R2204: value SELECT -> 0
- R1901: value 100k -> 10K; footprint Resistor_SMD:R_0603_1608Metric_Pad0.98x0.95mm_HandSolder -> Resistor_SMD:R_0603_1608Metric
- R1902: value 10K -> 39k
- R1903: value 39k -> 22
- R1904: value 22R -> 100
- R1905: value 100R -> 1k
- R1906: value 1k -> 150
- R1907: value 150R -> 2k49
- R204: value 36k -> 60k
- R205: value 40k -> 500k
- R206: value 60k -> 36k
- R211: value 67k -> 76k
- R212: value 100k -> 76k
- R213: value 1k -> 100k
- R214: value 10 -> 1k
- R901: value 100 -> 10
- R902: value 100 -> 100k
- U1401, U1402: value AP22653AW6-7 -> LM74700
- U1501: value TMCS1101A2UQDT -> TPS62933; footprint Package_SO:SOIC-8_3.9x4.9mm_P1.27mm -> Package_TO_SOT_SMD:SOT-583-8
- U1701: value AP22653AW6-7 -> TMCS1101A2UQDT; footprint Package_TO_SOT_SMD:SOT-23-6 -> Package_SO:SOIC-8_3.9x4.9mm_P1.27mm
- U401: value TMCS1101A2UQDT -> LM74700
- moved H104 219.2 mm to (243.1, 133.8)
- moved H102 212.8 mm to (240.5, 48.1)
- moved J109 192.8 mm to (212.4, 123.0), turned to 90 degrees
- moved J110 188.3 mm to (214.8, 103.3), turned to 90 degrees
- moved R105 179.5 mm to (206.2, 128.2), turned to 180 degrees
- moved C1703 168.6 mm to (237.0, 81.5), turned to 90 degrees
- moved J104 166.5 mm to (236.1, 132.8), turned to -90 degrees
- moved U1701 161.2 mm to (233.1, 79.8), turned to -90 degrees
- moved C1701 160.8 mm to (237.0, 77.9), turned to -90 degrees
- moved J107 154.0 mm to (177.9, 120.9), turned to 90 degrees
- moved C2006 150.5 mm to (240.5, 125.6), turned to 180 degrees
- moved R2104 150.2 mm to (233.7, 128.1), turned to -90 degrees
- moved J117 149.2 mm to (202.1, 58.1), turned to -90 degrees
- moved U2002 147.2 mm to (240.5, 122.8), turned to 0 degrees
- moved C2003 147.0 mm to (240.6, 99.7), turned to 180 degrees
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Connections:
- C1101 pad 1: /switch/Switch_element/VOUT1 -> /ameas/VIN
- C1102 pad 1: /switch/Switch_element/VOUT2 -> /ameas/VOUT
- C1103 pad 1: /switch/Switch_element/VOUT1 -> +5V
- C1103 pad 2: Net-(U1101-VCAP) -> GND
- C1104 pad 1: /switch/Switch_element/VOUT2 -> Net-(IC1102-ITIMER)
- C1104 pad 2: Net-(U1102-VCAP) -> GND
- C1105 pad 1: /switch/VOUT -> Net-(IC1101-DVDT)
- C1106 pad 1: /switch/VOUT -> Net-(IC1102-DVDT)
- C1401 pad 1: /switch_c/VIN -> /battery/Switch_Batt_Heater/VOUT1
- C1402 pad 1: /switch_c/VIN -> /battery/Switch_Batt_Heater/VOUT2
- C1403 pad 1: /switch_c/VOUT -> /battery/Switch_Batt_Heater/VOUT1
- C1403 pad 2: GND -> Net-(U1401-VCAP)
- C1404 pad 1: /switch_c/VOUT -> /battery/Switch_Batt_Heater/VOUT2
- C1404 pad 2: GND -> Net-(U1402-VCAP)
- C1501 pad 1: /ameas/VIN -> /dcdc/VIN
- C1502 pad 1: /ameas/VOUT -> /dcdc/VIN
- C1503 pad 1: +5V -> /dcdc/VIN
- C1701 pad 1: /solar/Switch_SOL_1/VIN1 -> /ameas/VIN
- C1702 pad 1: /solar/Switch_SOL_1/VIN1 -> /ameas/VOUT
- C1703 pad 1: /solar/Switch_SOL_1/Switch_element/VOUT1 -> +5V
- C1801 pad 1: /SOL_FIXED -> /switch_c/VIN
- C1802 pad 1: /SOL_FIXED -> /switch_c/VIN
- C1803 pad 1: /solar/Switch_SOL_2/Switch_element/VOUT1 -> Net-(IC1801-ITIMER)
- C1804 pad 1: /solar/Switch_SOL_2/Switch_element/VOUT2 -> Net-(IC1802-ITIMER)
- C201 pad 1: Net-(U201-VCC) -> Net-(U201-TERM_EN)
- C202 pad 1: Net-(U201-SRP) -> Net-(U201-VCC)
- C202 pad 2: /solar/Switch_SOL_1/VIN1 -> GND
- C203 pad 1: /solar/REGN -> Net-(U201-SRP)
- C203 pad 2: GND -> /solar/Switch_SOL_1/VIN1
- C204 pad 1: Net-(Q202-S) -> /solar/REGN
- C204 pad 2: Net-(D202-K) -> GND
- C205 pad 1: Net-(D201-K) -> Net-(Q202-S)
- C205 pad 2: GND -> Net-(D202-K)
- C206 pad 1: /solar/Switch_SOL_1/VIN1 -> Net-(D201-K)
- C207 pad 2: Net-(U201-VFB) -> GND
- C208 pad 2: GND -> Net-(U201-VFB)
- C2101 pad 1: /Battery -> /battery/BATT
- C2102 pad 1: /Battery -> /battery/BATT
- C2103 pad 1: /battery/Switch_Batt_Heater/Switch_element/VOUT1 -> Net-(IC2101-ITIMER)
- C2104 pad 1: /battery/Switch_Batt_Heater/Switch_element/VOUT2 -> Net-(IC2102-ITIMER)
- C2203 pad 1: /switch/Switch_element/VOUT1 -> Net-(IC2201-ITIMER)
- C2204 pad 1: /switch/Switch_element/VOUT2 -> Net-(IC2202-ITIMER)
- C401 pad 1: /PV -> /solar/Switch_SOL_1/VOUT1
- C402 pad 1: /solar/PV -> /solar/Switch_SOL_1/VOUT2
- C403 pad 1: +5V -> /solar/Switch_SOL_1/VOUT1
- C403 pad 2: GND -> Net-(U401-VCAP)
- J102 pad 1: GND -> /solar/Enable
- J102 pad 2: /battery/HEATER -> /SOL_STAT_2
- J102 pad 3: (no net) -> /SOL_STAT_1
- J102 pad 4: (no net) -> unconnected-(J102-Pin_4-Pad4)
- J103 pad 1: /Battery -> GND
- J104 pad 1: /HEAT_BATT_1 -> /battery/HEATER
- J104 pad 2: /SWITCH_EN -> GND
- J105 pad 1: Net-(J105-Pin_1) -> GND
- J105 pad 2: GND -> /MPPT_~{EN}
- J105 pad 3: (no net) -> +5V
- J107 pad 1: /dcdc/EN -> /solar/AMEAS
- J107 pad 2: /dcdc/VIN -> /TMEAS
- J107 pad 3: (no net) -> /solar/VMEAS
- J109 pad 1: GND -> /solar/VOUT
- J109 pad 2: /Ch_EN_12 -> GND
- J110 pad 1: /switch_c/VOUT -> GND
- J111 pad 1: /ameas/VIN -> /solar/VOUT
- J111 pad 2: GND -> /Battery
- J116 pad 1: GND -> /switch/VIN1
- J116 pad 2: /AMEAS_1 -> GND
- J117 pad 1: /ameas/VOUT -> /ameas1/AMEAS
- Q1901 pad 3: /battery/Temp_sens_battery/Curr_source -> /battery/CC_Source/CC_Source
- R105 pad 1: /switch/VOUT -> /Battery
- R105 pad 2: /dcdc/VIN -> /battery/BATT
- R1401 pad 1: /Ch_AL_1 -> GND
- R1401 pad 2: /switch_c/VIN -> /battery/Heater_EN
- R1801 pad 1: /solar/Switch_SOL_2/~{ALERT} -> GND
- R1801 pad 2: /SOL_FIXED -> /Ch_EN_11
- R1802 pad 1: /solar/Switch_SOL_2/~{ALERT} -> GND
- R1802 pad 2: /SOL_FIXED -> /Ch_EN_12
- R1901 pad 1: /TMEAS_BATT_1 -> Net-(U1901-IN+)
- R1901 pad 2: /battery/Temp_sens_battery/Curr_source -> +3V3
- R1902 pad 1: Net-(U1901-IN+) -> GND
- R1902 pad 2: +3V3 -> Net-(U1901-IN+)
- R1903 pad 1: GND -> Net-(U1901-EN)
- R1903 pad 2: Net-(U1901-IN+) -> +3V3
- R1904 pad 1: Net-(U1901-EN) -> Net-(Q1901-G)
- R1904 pad 2: +3V3 -> Net-(U1901-OUT)
- R1905 pad 1: Net-(Q1901-G) -> Net-(Q1901-S)
- R1905 pad 2: Net-(U1901-OUT) -> Net-(U1901-IN-)
- R1906 pad 1: Net-(Q1901-S) -> Net-(R1906-Pad1)
- R1906 pad 2: Net-(U1901-IN-) -> +3V3
- R1907 pad 1: Net-(R1907-Pad1) -> Net-(Q1901-S)
- R1907 pad 2: +3V3 -> Net-(R1906-Pad1)
- R201 pad 2: /VMEAS_SOL_1 -> /solar/VMEAS
- R202 pad 1: /VMEAS_SOL_1 -> /solar/VMEAS
- R204 pad 1: Net-(Q201-D) -> /solar/Term
- R205 pad 1: Net-(U201-TERM_EN) -> /solar/PV
- R205 pad 2: /solar/Term -> Net-(Q201-D)
- R206 pad 1: /solar/Term -> Net-(Q201-D)
- R2101 pad 1: /battery/Switch_Batt_Heater/~{ALERT} -> GND
- R2101 pad 2: /Battery -> /battery/Heater_EN
- R2102 pad 1: /battery/Switch_Batt_Heater/~{ALERT} -> GND
- R2102 pad 2: /Battery -> /battery/Heater_EN
- R212 pad 1: /solar/Switch_SOL_1/EN -> Net-(U201-VFB)
- R212 pad 2: /solar/Switch_SOL_1/VIN1 -> GND
- R213 pad 1: /SOL_TGGL_1 -> /solar/Switch_SOL_1/EN
- R213 pad 2: /solar/Switch_SOL_1/EN -> /solar/Switch_SOL_1/VIN1
- R214 pad 1: Net-(Q204-G) -> /SOL_TGGL
- R214 pad 2: /SOL_TGGL_1 -> /solar/Switch_SOL_1/EN
- R2201 pad 1: /SWITCH_ALERT -> GND
- R2201 pad 2: /switch/VIN1 -> /SW_EN
- R2202 pad 1: /SWITCH_ALERT -> GND
- R2202 pad 2: /switch/VIN1 -> /SW_EN
- R901 pad 1: /battery/VC5 -> Net-(Q902-S)
- R901 pad 2: /Battery -> Net-(Q901-G)
- R902 pad 1: /battery/BATT_3 -> /dcdc/VIN
- R902 pad 2: /battery/VC3 -> Net-(Q901-S)
- TP201 pad 1: /solar/PV -> /solar/Term
- TP202 pad 1: /solar/Term -> /solar/PV
- TP205 pad 1: /SOL_TGGL_1 -> /SOL_TGGL
- U1401 pad 1: /switch_c/VOUT -> Net-(U1401-VCAP)
- U1401 pad 3: /Ch_EN_11 -> /battery/Switch_Batt_Heater/VOUT1
- U1401 pad 4: /Ch_AL_1 -> /battery/HEATER
- U1401 pad 6: /switch_c/VIN -> /battery/Switch_Batt_Heater/VOUT1
- U1402 pad 1: /switch_c/VOUT -> Net-(U1402-VCAP)
- U1402 pad 3: /Ch_EN_12 -> /battery/Switch_Batt_Heater/VOUT2
- U1402 pad 4: /Ch_AL_1 -> /battery/HEATER
- U1402 pad 6: /switch_c/VIN -> /battery/Switch_Batt_Heater/VOUT2
- U1501 pad 1: /ameas/VIN -> Net-(U1501-RT)
- U1501 pad 2: /ameas/VIN -> /dcdc/EN
- U1501 pad 3: /ameas/VOUT -> /dcdc/VIN
- U1501 pad 4: /ameas/VOUT -> GND
- U1501 pad 5: GND -> Net-(U1501-SW)
- U1501 pad 6: unconnected-(U1501-BW_SEL-Pad6) -> Net-(U1501-BST)
- U1501 pad 7: /AMEAS_1 -> Net-(U1501-SS)
- U1501 pad 8: +5V -> Net-(U1501-FB)
- U1701 pad 1: /solar/Switch_SOL_1/Switch_element/VOUT1 -> /ameas/VIN
- U1701 pad 2: GND -> /ameas/VIN
- U1701 pad 3: /solar/Switch_SOL_1/EN -> /ameas/VOUT
- U1701 pad 4: /solar/Switch_SOL_1/~{ALERT} -> /ameas/VOUT
- U1701 pad 5: Net-(U1701-ISET) -> GND
- U1701 pad 6: /solar/Switch_SOL_1/VIN1 -> unconnected-(U1701-BW_SEL-Pad6)
- U401 pad 1: /PV -> Net-(U401-VCAP)
- U401 pad 2: /PV -> GND
- U401 pad 3: /solar/PV -> /solar/Switch_SOL_1/VOUT1
- U401 pad 4: /solar/PV -> /solar/VOUT
- U401 pad 5: GND -> Net-(Q401-G)
- U401 pad 6: unconnected-(U401-BW_SEL-Pad6) -> /solar/Switch_SOL_1/VOUT1
- U401 pad 7: /AMEAS_SOL_1 -> (no net)
- U401 pad 8: +5V -> (no net)
Routing:
- net /battery/BATT: track 0.00 -> 168.9 mm
- net +5V: track 3.21 -> 170.4 mm, vias 2 -> 3
- net +3V3: track 0.00 -> 135.0 mm
- net /solar/PV: track 82.1 -> 17.8 mm, vias 2 -> 0
- net Net-(Q1502-S): track 0.00 -> 62.1 mm
- net Net-(Q502-S): track 54.7 -> 0.00 mm
- net GND: track 24.9 -> 74.0 mm, vias 133 -> 193
- net Net-(Q1202-S): track 45.5 -> 0.00 mm
- net /SOL_TGGL_1: track 45.2 -> 0.00 mm, vias 1 -> 0
- net /SOL_FIXED: track 44.2 -> 0.00 mm, vias 5 -> 0
- net /switch_c/VIN: track 9.08 -> 52.3 mm
- net /battery/Heater_EN: track 0.00 -> 40.2 mm, vias 0 -> 2
- net /SWITCH_EN: track 39.5 -> 0.00 mm, vias 4 -> 0
- net /dcdc/VOUT: track 0.00 -> 38.1 mm
- net /solar/VOUT: track 92.3 -> 54.6 mm, vias 16 -> 0
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Other:
- board size 90 x 95.8 mm -> 181.4 x 95.8 mm
