File: CC_SOURCE_SIMPLE.kicad_sch (KiCad schematic)
At the start: 3 parts, among them U501 LM334M

Commit message: nearly finnished CORE pcb
Parts:
- renumbered R501 to R6502, U501 to U6501
Changed lines of the file:
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@@
 		(dnp no)
 		(fields_autoplaced yes)
-		(property "Reference" "U501"
+		(property "Reference" "U6501"
 			(at 158.75 92.3924 0)
 			(effects
@@
 		(dnp no)
 		(fields_autoplaced yes)
-		(property "Reference" "#PWR0501"
+		(property "Reference" "#PWR?"
 			(at 144.78 97.79 0)
 			(effects
@@
 				(path "/29496ace-b476-4f24-a65f-9da1dd70122c/e4dfe94c-1781-4e0e-8290-73a1da958379/f372b097-c94b-4e63-a97a-bb43e24599a8"
 					(reference "#PWR0501")
+					(unit 1)
+				)
+			)
+			(project "EPS"
+				(path "/94201994-47b8-4213-8d1a-05da12b2a7b0/f14e2ccd-368c-4564-a2f9-aaa88b448b60/f372b097-c94b-4e63-a97a-bb43e24599a8"
+					(reference "#PWR?")
 					(unit 1)
 				)
@@
 		(dnp no)
 		(fields_autoplaced yes)
-		(property "Reference" "C501"
+		(property "Reference" "C?"
 			(at 147.32 87.6362 0)
 			(effects
@@
 				(path "/29496ace-b476-4f24-a65f-9da1dd70122c/e4dfe94c-1781-4e0e-8290-73a1da958379/f372b097-c94b-4e63-a97a-bb43e24599a8"
 					(reference "C501")
+					(unit 1)
+				)
+			)
+			(project "EPS"
+				(path "/94201994-47b8-4213-8d1a-05da12b2a7b0/f14e2ccd-368c-4564-a2f9-aaa88b448b60/f372b097-c94b-4e63-a97a-bb43e24599a8"
+					(reference "C?")
 					(unit 1)
 				)
@@
 		(dnp no)
 		(fields_autoplaced yes)
-		(property "Reference" "R501"
+		(property "Reference" "R6502"
 			(at 170.18 96.5199 0)
 			(effects
