File: MCU.kicad_sch (KiCad schematic)
At the start: 86 parts, among them J901 Conn_01x02_Pin, J902 JTAG, J903 JTAG, U901 LP38690SDX-3.3/NOPB, U902 MSP430FR5969IRGZR, U903 ADG1607xCP, U904 MSP430FR5969IRGZR, U905 TCAN4551RGYRQ1, U906 ADG1607xCP, Y901 Crystal, Y902 Crystal

Commit message: small changes to test board
Parts:
- renumbered C926 to C1225, C925 to C1226, C911 to C1227, C912 to C1228, C901 to C1229, C914 to C1230, C920 to C1231, C928 to C1232, C931 to C1233, C927 to C1234, C913 to C1235, C906 to C1236, C908 to C1237, C915 to C1238, C917 to C1239, C907 to C1240, C909 to C1241, C916 to C1242, C918 to C1243, C910 to C1244, C919 to C1245, C922 to C1246, C924 to C1247, C929 to C1248, C902 to C1302, C905 to C1307, C903 to C1308, C904 to C1309, C921 to C1322, C930 to C1325, C923 to C1326, J902 to J1201, J903 to J1202, J901 to J1301, R917 to R1210, R901 to R1211, R902 to R1212, R904 to R1213, R907 to R1214, R910 to R1215, R913 to R1216, R914 to R1217, R905 to R1218, R908 to R1219, R911 to R1220, R906 to R1221, R909 to R1222, R912 to R1223, R918 to R1224, R922 to R1225, R921 to R1226, R916 to R1227, R903 to R1228, R919 to R1229, R915 to R1309, R920 to R1319, R923 to R1320, R924 to R1321, R_MISO_901 to R_MISO_1201, R_MOSI_901 to R_MOSI_1201, R_RX_901 to R_RX_1201, R_TX_901 to R_TX_1201, TP910 to TP1201, TP911 to TP1202, TP912 to TP1203, TP913 to TP1204, TP917 to TP1205, TP914 to TP1206, TP916 to TP1207, TP901 to TP1301, TP903 to TP1302, TP904 to TP1303, TP902 to TP1306, TP915 to TP1311, TP905 to TP1315, TP906 to TP1316, TP908 to TP1317, TP907 to TP1318, U903 to U1205, U906 to U1206, U905 to U1207, U901 to U1303, U902 to U1304, U904 to U1305, Y902 to Y1201, Y901 to Y1202

Commit message: nearly finnished CORE pcb
Parts:
- C920: renamed from C1231; now not fitted; now left out of the parts list
- C931: renamed from C1233; now not fitted; now left out of the parts list
- J902: renamed from J1201; symbol Connector:Conn_01x04_Socket -> Connector_Generic_MountingPin:Conn_01x04_MountingPin
- J903: renamed from J1202; symbol Connector:Conn_01x04_Socket -> Connector_Generic_MountingPin:Conn_01x04_MountingPin
- renumbered C1229 to C901, C1302 to C902, C1308 to C903, C1309 to C904, C1307 to C905, C1236 to C906, C1240 to C907, C1237 to C908, C1241 to C909, C1244 to C910, C1227 to C911, C1228 to C912, C1235 to C913, C1230 to C914, C1238 to C915, C1242 to C916, C1239 to C917, C1243 to C918, C1245 to C919, C1322 to C921, C1246 to C922, C1326 to C923, C1247 to C924, C1226 to C925, C1225 to C926, C1234 to C927, C1232 to C928, C1248 to C929, C1325 to C930, J1301 to J901, R1211 to R901, R1212 to R902, R1228 to R903, R1213 to R904, R1218 to R905, R1221 to R906, R1214 to R907, R1219 to R908, R1222 to R909, R1215 to R910, R1220 to R911, R1223 to R912, R1216 to R913, R1217 to R914, R1309 to R915, R1227 to R916, R1210 to R917, R1224 to R918, R1229 to R919, R1319 to R920, R1226 to R921, R1225 to R922, R1320 to R923, R1321 to R924, R_MISO_1201 to R_MISO_901, R_MOSI_1201 to R_MOSI_901, R_RX_1201 to R_RX_901, R_TX_1201 to R_TX_901, TP1301 to TP901, TP1306 to TP902, TP1302 to TP903, TP1303 to TP904, TP1315 to TP905, TP1316 to TP906, TP1318 to TP907, TP1317 to TP908, TP1201 to TP910, TP1202 to TP911, TP1203 to TP912, TP1204 to TP913, TP1206 to TP914, TP1311 to TP915, TP1207 to TP916, TP1205 to TP917, U1303 to U901, U1304 to U902, U1205 to U903, U1305 to U904, U1207 to U905, U1206 to U906, Y1202 to Y901, Y1201 to Y902
Connections:
- net ADC_3: now also U902.9 (P1.3/TA1.2/UCB0STE/A3/C3); no longer U902.3 (P1.2/TA1.1/TA0CLK/COUT/A2/C2)
- net ADC_4: now also U902.3 (P1.2/TA1.1/TA0CLK/COUT/A2/C2); no longer U902.9 (P1.3/TA1.2/UCB0STE/A3/C3)
- net AMEAS_10: now also U906.7 (S2B); no longer U903.7 (S2B)
- net AMEAS_2: no longer TP910.1, U906.19 (S3A)
- net AMEAS_9: no longer TP914.1, U903.8 (S1B)
- net AMUX_0: now also U902.34 (P4.5); no longer U902.33 (P4.4/TB0.5)
- net AMUX_1: now also U902.35 (P4.6); no longer U902.34 (P4.5)
- net AMUX_2: now also U902.39 (P2.3/TA0.0/UCA1STE/A6/C10); no longer U902.35 (P4.6)
- net AMUX_EN: now also U902.33 (P4.4/TB0.5); no longer U902.39 (P2.3/TA0.0/UCA1STE/A6/C10)
- net BATT_ALERT_1: now also U902.7 (P3.3/A15/C15); no longer U902.6 (P3.2/A14/C14)
- net BATT_ALERT_2: now also U902.6 (P3.2/A14/C14); no longer U902.7 (P3.3/A15/C15)
- net TMEAS_BATT_2: now also U903.7 (S2B); no longer U906.7 (S2B)
- new net SHIELD: J902.MP (MountPin), J903.MP (MountPin)
- new net TMEAS_BATT_1: TP914.1, U903.8 (S1B)
- new net VMEAS_SOL_1: TP910.1, U906.19 (S3A)
Other:
- sheet RS422_485 ports: added A_N, B_P; removed A_P, B_N

Commit message: pcb progres for all components
Parts:
- renumbered C926 to C1225, C925 to C1226, C911 to C1227, C912 to C1228, C901 to C5001, C902 to C5002, C914 to C5003, C920 to C5004, C928 to C5005, C931 to C5006, C905 to C5007, C903 to C5008, C904 to C5009, C927 to C5011, C913 to C5012, C906 to C5013, C908 to C5014, C915 to C5015, C917 to C5016, C907 to C5017, C909 to C5018, C916 to C5019, C918 to C5020, C910 to C5021, C919 to C5022, C921 to C5023, C922 to C5024, C924 to C5025, C930 to C5026, C923 to C5027, C929 to C5028, J901 to J1301, J902 to J5002, J903 to J5004, R917 to R1210, R901 to R1211, R902 to R1212, R914 to R5001, R904 to R5002, R907 to R5003, R910 to R5004, R913 to R5005, R915 to R5006, R905 to R5007, R908 to R5008, R911 to R5009, R906 to R5010, R909 to R5011, R912 to R5012, R918 to R5013, R922 to R5014, R921 to R5016, R916 to R5017, R903 to R5018, R919 to R5019, R920 to R5020, R923 to R5021, R924 to R5022, R_MISO_901 to R_MISO_5001, R_MOSI_901 to R_MOSI_5001, R_RX_901 to R_RX_5001, R_TX_901 to R_TX_5001, TP903 to TP1302, TP904 to TP1303, TP905 to TP1315, TP906 to TP1316, TP908 to TP1317, TP907 to TP1318, TP901 to TP5001, TP902 to TP5002, TP910 to TP5003, TP911 to TP5004, TP912 to TP5005, TP913 to TP5006, TP915 to TP5007, TP917 to TP5008, TP914 to TP5009, TP916 to TP5010, U903 to U5001, U906 to U5002, U901 to U5003, U902 to U5004, U904 to U5005, U905 to U5006, Y902 to Y1201, Y901 to Y1202
