File: RS422_485.kicad_sch (KiCad schematic)
At the start: 10 parts, among them U401 THVD1424

Commit message: progress on CORE pcb
Parts:
- renumbered C401 to C1101, JP401 to JP1101, JP402 to JP1102, R402 to R1101, R403 to R1102, R404 to R1103, R405 to R1104, R406 to R1105, R401 to R1106, U401 to U1101
Changed lines of the file:
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@@
 		(on_board yes)
 		(dnp no)
-		(property "Reference" "R405"
+		(property "Reference" "R1104"
 			(at 208.28 97.7899 0)
 			(effects
@@
 		(instances
 			(project "EPS_CORE"
-				(path "/29496ace-b476-4f24-a65f-9da1dd70122c/59fca87d-eab6-4325-93c7-8130e49f891e/6fcf384b-60b0-45a5-8dc1-cf23d8e5c23c"
-					(reference "R405")
-					(unit 1)
-				)
-			)
-			(project "EPS_CORE"
 				(path "/43e5e7c8-e7e0-4528-9a3e-b1557849918d/ce55ed75-3d20-4bd3-84d2-d62dbd0d02de/6fcf384b-60b0-45a5-8dc1-cf23d8e5c23c"
-					(reference "R?")
+					(reference "R1104")
 					(unit 1)
 				)
@@
 		(on_board yes)
 		(dnp no)
-		(property "Reference" "R403"
+		(property "Reference" "R1102"
 			(at 163.83 85.725 0)
 			(effects
@@
 		(instances
 			(project "EPS_CORE"
-				(path "/29496ace-b476-4f24-a65f-9da1dd70122c/59fca87d-eab6-4325-93c7-8130e49f891e/6fcf384b-60b0-45a5-8dc1-cf23d8e5c23c"
-					(reference "R403")
-					(unit 1)
-				)
-			)
-			(project "EPS_CORE"
 				(path "/43e5e7c8-e7e0-4528-9a3e-b1557849918d/ce55ed75-3d20-4bd3-84d2-d62dbd0d02de/6fcf384b-60b0-45a5-8dc1-cf23d8e5c23c"
-					(reference "R?")
+					(reference "R1102")
 					(unit 1)
 				)
@@
 		(dnp yes)
 		(fields_autoplaced yes)
-		(property "Reference" "JP401"
+		(property "Reference" "JP1101"
 			(at 121.92 91.44 90)
 			(effects
@@
 		(instances
 			(project "EPS_CORE"
-				(path "/29496ace-b476-4f24-a65f-9da1dd70122c/59fca87d-eab6-4325-93c7-8130e49f891e/6fcf384b-60b0-45a5-8dc1-cf23d8e5c23c"
-					(reference "JP401")
-					(unit 1)
-				)
-			)
-			(project "EPS_CORE"
 				(path "/43e5e7c8-e7e0-4528-9a3e-b1557849918d/ce55ed75-3d20-4bd3-84d2-d62dbd0d02de/6fcf384b-60b0-45a5-8dc1-cf23d8e5c23c"
-					(reference "JP?")
+					(reference "JP1101")
 					(unit 1)
 				)
@@
 		(on_board yes)
 		(dnp no)
-		(property "Reference" "#PWR0403"
+		(property "Reference" "#PWR0328"
 			(at 142.24 125.73 0)
 			(effects
@@
 		(instances
 			(project "EPS_CORE"
-				(path "/29496ace-b476-4f24-a65f-9da1dd70122c/59fca87d-eab6-4325-93c7-8130e49f891e/6fcf384b-60b0-45a5-8dc1-cf23d8e5c23c"
-					(reference "#PWR0403")
-					(unit 1)
-				)
-			)
-			(project "EPS_CORE"
 				(path "/43e5e7c8-e7e0-4528-9a3e-b1557849918d/ce55ed75-3d20-4bd3-84d2-d62dbd0d02de/6fcf384b-60b0-45a5-8dc1-cf23d8e5c23c"
-					(reference "#PWR?")
+					(reference "#PWR0328")
 					(unit 1)
 				)
@@
 		(dnp no)
 		(fields_autoplaced yes)
-		(property "Reference" "C401"
+		(property "Reference" "C1101"
 			(at 137.16 80.0035 0)
 			(effects
@@
 		(instances
 			(project "EPS_CORE"
-				(path "/29496ace-b476-4f24-a65f-9da1dd70122c/59fca87d-eab6-4325-93c7-8130e49f891e/6fcf384b-60b0-45a5-8dc1-cf23d8e5c23c"
-					(reference "C401")
-					(unit 1)
-				)
-			)
-			(project "EPS_CORE"
 				(path "/43e5e7c8-e7e0-4528-9a3e-b1557849918d/ce55ed75-3d20-4bd3-84d2-d62dbd0d02de/6fcf384b-60b0-45a5-8dc1-cf23d8e5c23c"
-					(reference "C?")
+					(reference "C1101")
 					(unit 1)
 				)
@@
 		(dnp no)
 		(fields_autoplaced yes)
-		(property "Reference" "R402"
+		(property "Reference" "R1101"
 			(at 148.59 85.09 0)
 			(effects
@@
 		(instances
 			(project "EPS_CORE"
-				(path "/29496ace-b476-4f24-a65f-9da1dd70122c/59fca87d-eab6-4325-93c7-8130e49f891e/6fcf384b-60b0-45a5-8dc1-cf23d8e5c23c"
-					(reference "R402")
-					(unit 1)
-				)
-			)
-			(project "EPS_CORE"
 				(path "/43e5e7c8-e7e0-4528-9a3e-b1557849918d/ce55ed75-3d20-4bd3-84d2-d62dbd0d02de/6fcf384b-60b0-45a5-8dc1-cf23d8e5c23c"
-					(reference "R?")
+					(reference "R1101")
 					(unit 1)
 				)
@@
 		(on_board yes)
 		(dnp no)
-		(property "Reference" "#PWR0405"
+		(property "Reference" "#PWR0324"
 			(at 189.23 128.27 0)
 			(effects
@@
 		(instances
 			(project "EPS_CORE"
-				(path "/29496ace-b476-4f24-a65f-9da1dd70122c/59fca87d-eab6-4325-93c7-8130e49f891e/6fcf384b-60b0-45a5-8dc1-cf23d8e5c23c"
-					(reference "#PWR0405")
-					(unit 1)
-				)
-			)
-			(project "EPS_CORE"
 				(path "/43e5e7c8-e7e0-4528-9a3e-b1557849918d/ce55ed75-3d20-4bd3-84d2-d62dbd0d02de/6fcf384b-60b0-45a5-8dc1-cf23d8e5c23c"
-					(reference "#PWR?")
+					(reference "#PWR0324")
 					(unit 1)
 				)
@@
 		(dnp no)
 		(fields_autoplaced yes)
-		(property "Reference" "R404"
+		(property "Reference" "R1103"
 			(at 173.99 85.09 0)
 			(effects
@@
 		(instances
 			(project "EPS_CORE"
-				(path "/29496ace-b476-4f24-a65f-9da1dd70122c/59fca87d-eab6-4325-93c7-8130e49f891e/6fcf384b-60b0-45a5-8dc1-cf23d8e5c23c"
-					(reference "R404")
-					(unit 1)
-				)
-			)
-			(project "EPS_CORE"
 				(path "/43e5e7c8-e7e0-4528-9a3e-b1557849918d/ce55ed75-3d20-4bd3-84d2-d62dbd0d02de/6fcf384b-60b0-45a5-8dc1-cf23d8e5c23c"
-					(reference "R?")
+					(reference "R1103")
 					(unit 1)
 				)
@@
 		(on_board yes)
 		(dnp no)
-		(property "Reference" "#PWR0401"
+		(property "Reference" "#PWR0327"
 			(at 110.49 109.22 0)
 			(effects
@@
 		(instances
 			(project "EPS_CORE"
-				(path "/29496ace-b476-4f24-a65f-9da1dd70122c/59fca87d-eab6-4325-93c7-8130e49f891e/6fcf384b-60b0-45a5-8dc1-cf23d8e5c23c"
-					(reference "#PWR0401")
-					(unit 1)
-				)
-			)
-			(project "EPS_CORE"
 				(path "/43e5e7c8-e7e0-4528-9a3e-b1557849918d/ce55ed75-3d20-4bd3-84d2-d62dbd0d02de/6fcf384b-60b0-45a5-8dc1-cf23d8e5c23c"
-					(reference "#PWR?")
+					(reference "#PWR0327")
 					(unit 1)
 				)
@@
 		(dnp no)
 		(fields_autoplaced yes)
-		(property "Reference" "R401"
+		(property "Reference" "R1106"
 			(at 139.7 114.2999 0)
 			(effects
@@
 		(instances
 			(project "EPS_CORE"
-				(path "/29496ace-b476-4f24-a65f-9da1dd70122c/59fca87d-eab6-4325-93c7-8130e49f891e/6fcf384b-60b0-45a5-8dc1-cf23d8e5c23c"
-					(reference "R401")
-					(unit 1)
-				)
-			)
-			(project "EPS_CORE"
 				(path "/43e5e7c8-e7e0-4528-9a3e-b1557849918d/ce55ed75-3d20-4bd3-84d2-d62dbd0d02de/6fcf384b-60b0-45a5-8dc1-cf23d8e5c23c"
-					(reference "R?")
+					(reference "R1106")
 					(unit 1)
 				)
@@
 		(dnp no)
 		(fields_autoplaced yes)
-		(property "Reference" "U401"
+		(property "Reference" "U1101"
 			(at 190.1541 86.36 0)
 			(effects
@@
 		(instances
 			(project "EPS_CORE"
-				(path "/29496ace-b476-4f24-a65f-9da1dd70122c/59fca87d-eab6-4325-93c7-8130e49f891e/6fcf384b-60b0-45a5-8dc1-cf23d8e5c23c"
-					(reference "U401")
-					(unit 1)
-				)
-			)
-			(project "EPS_CORE"
 				(path "/43e5e7c8-e7e0-4528-9a3e-b1557849918d/ce55ed75-3d20-4bd3-84d2-d62dbd0d02de/6fcf384b-60b0-45a5-8dc1-cf23d8e5c23c"
-					(reference "U?")
+					(reference "U1101")
 					(unit 1)
 				)
@@
 		(on_board yes)
 		(dnp no)
-		(property "Reference" "#PWR0404"
+		(property "Reference" "#PWR0325"
 			(at 176.53 128.27 0)
 			(effects
@@
 		(instances
 			(project "EPS_CORE"
-				(path "/29496ace-b476-4f24-a65f-9da1dd70122c/59fca87d-eab6-4325-93c7-8130e49f891e/6fcf384b-60b0-45a5-8dc1-cf23d8e5c23c"
-					(reference "#PWR0404")
-					(unit 1)
-				)
-			)
-			(project "EPS_CORE"
 				(path "/43e5e7c8-e7e0-4528-9a3e-b1557849918d/ce55ed75-3d20-4bd3-84d2-d62dbd0d02de/6fcf384b-60b0-45a5-8dc1-cf23d8e5c23c"
-					(reference "#PWR?")
+					(reference "#PWR0325")
 					(unit 1)
 				)
@@
 		(on_board yes)
 		(dnp no)
-		(property "Reference" "R406"
+		(property "Reference" "R1105"
 			(at 208.28 107.9499 0)
 			(effects
@@
 		(instances
 			(project "EPS_CORE"
-				(path "/29496ace-b476-4f24-a65f-9da1dd70122c/59fca87d-eab6-4325-93c7-8130e49f891e/6fcf384b-60b0-45a5-8dc1-cf23d8e5c23c"
-					(reference "R406")
-					(unit 1)
-				)
-			)
-			(project "EPS_CORE"
 				(path "/43e5e7c8-e7e0-4528-9a3e-b1557849918d/ce55ed75-3d20-4bd3-84d2-d62dbd0d02de/6fcf384b-60b0-45a5-8dc1-cf23d8e5c23c"
-					(reference "R?")
+					(reference "R1105")
 					(unit 1)
 				)
@@
 		(on_board yes)
 		(dnp no)
-		(property "Reference" "#PWR0402"
+		(property "Reference" "#PWR0326"
 			(at 139.7 90.17 0)
 			(effects
@@
 		(instances
 			(project "EPS_CORE"
-				(path "/29496ace-b476-4f24-a65f-9da1dd70122c/59fca87d-eab6-4325-93c7-8130e49f891e/6fcf384b-60b0-45a5-8dc1-cf23d8e5c23c"
-					(reference "#PWR0402")
-					(unit 1)
-				)
-			)
-			(project "EPS_CORE"
 				(path "/43e5e7c8-e7e0-4528-9a3e-b1557849918d/ce55ed75-3d20-4bd3-84d2-d62dbd0d02de/6fcf384b-60b0-45a5-8dc1-cf23d8e5c23c"
-					(reference "#PWR?")
+					(reference "#PWR0326")
 					(unit 1)
 				)
@@
 		(dnp yes)
 		(fields_autoplaced yes)
-		(property "Reference" "JP402"
+		(property "Reference" "JP1102"
 			(at 130.81 100.33 0)
 			(effects
@@
 		(instances
 			(project "EPS_CORE"
-				(path "/29496ace-b476-4f24-a65f-9da1dd70122c/59fca87d-eab6-4325-93c7-8130e49f891e/6fcf384b-60b0-45a5-8dc1-cf23d8e5c23c"
-					(reference "JP402")
-					(unit 1)
-				)
-			)
-			(project "EPS_CORE"
 				(path "/43e5e7c8-e7e0-4528-9a3e-b1557849918d/ce55ed75-3d20-4bd3-84d2-d62dbd0d02de/6fcf384b-60b0-45a5-8dc1-cf23d8e5c23c"
-					(reference "JP?")
-					(unit 1)
-				)
+					(reference "JP1102")
+					(unit 1)
+				)

Commit message: small changes to test board
Parts:
- renumbered C1101 to C401, JP1101 to JP401, JP1102 to JP402, R1106 to R401, R1101 to R402, R1102 to R403, R1103 to R404, R1104 to R405, R1105 to R406, U1101 to U401
Changed lines of the file:
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@@
 		(on_board yes)
 		(dnp no)
-		(property "Reference" "R1104"
+		(property "Reference" "R405"
 			(at 208.28 97.7899 0)
 			(effects
@@
 		)
 		(instances
+			(project "TEST_PCB"
+				(path "/29496ace-b476-4f24-a65f-9da1dd70122c/59fca87d-eab6-4325-93c7-8130e49f891e/6fcf384b-60b0-45a5-8dc1-cf23d8e5c23c"
+					(reference "R405")
+					(unit 1)
+				)
+			)
 			(project "EPS_CORE"
 				(path "/43e5e7c8-e7e0-4528-9a3e-b1557849918d/ce55ed75-3d20-4bd3-84d2-d62dbd0d02de/6fcf384b-60b0-45a5-8dc1-cf23d8e5c23c"
@@
 		(on_board yes)
 		(dnp no)
-		(property "Reference" "R1102"
+		(property "Reference" "R403"
 			(at 163.83 85.725 0)
 			(effects
@@
 		)
 		(instances
+			(project "TEST_PCB"
+				(path "/29496ace-b476-4f24-a65f-9da1dd70122c/59fca87d-eab6-4325-93c7-8130e49f891e/6fcf384b-60b0-45a5-8dc1-cf23d8e5c23c"
+					(reference "R403")
+					(unit 1)
+				)
+			)
 			(project "EPS_CORE"
 				(path "/43e5e7c8-e7e0-4528-9a3e-b1557849918d/ce55ed75-3d20-4bd3-84d2-d62dbd0d02de/6fcf384b-60b0-45a5-8dc1-cf23d8e5c23c"
@@
 		(dnp yes)
 		(fields_autoplaced yes)
-		(property "Reference" "JP1101"
+		(property "Reference" "JP401"
 			(at 121.92 91.44 90)
 			(effects
@@
 		)
 		(instances
+			(project "TEST_PCB"
+				(path "/29496ace-b476-4f24-a65f-9da1dd70122c/59fca87d-eab6-4325-93c7-8130e49f891e/6fcf384b-60b0-45a5-8dc1-cf23d8e5c23c"
+					(reference "JP401")
+					(unit 1)
+				)
+			)
 			(project "EPS_CORE"
 				(path "/43e5e7c8-e7e0-4528-9a3e-b1557849918d/ce55ed75-3d20-4bd3-84d2-d62dbd0d02de/6fcf384b-60b0-45a5-8dc1-cf23d8e5c23c"
@@
 		(on_board yes)
 		(dnp no)
-		(property "Reference" "#PWR0328"
+		(property "Reference" "#PWR0172"
 			(at 142.24 125.73 0)
 			(effects
@@
 		)
 		(instances
+			(project "TEST_PCB"
+				(path "/29496ace-b476-4f24-a65f-9da1dd70122c/59fca87d-eab6-4325-93c7-8130e49f891e/6fcf384b-60b0-45a5-8dc1-cf23d8e5c23c"
+					(reference "#PWR0172")
+					(unit 1)
+				)
+			)
 			(project "EPS_CORE"
 				(path "/43e5e7c8-e7e0-4528-9a3e-b1557849918d/ce55ed75-3d20-4bd3-84d2-d62dbd0d02de/6fcf384b-60b0-45a5-8dc1-cf23d8e5c23c"
@@
 		(dnp no)
 		(fields_autoplaced yes)
-		(property "Reference" "C1101"
+		(property "Reference" "C401"
 			(at 137.16 80.0035 0)
 			(effects
@@
 		)
 		(instances
+			(project "TEST_PCB"
+				(path "/29496ace-b476-4f24-a65f-9da1dd70122c/59fca87d-eab6-4325-93c7-8130e49f891e/6fcf384b-60b0-45a5-8dc1-cf23d8e5c23c"
+					(reference "C401")
+					(unit 1)
+				)
+			)
 			(project "EPS_CORE"
 				(path "/43e5e7c8-e7e0-4528-9a3e-b1557849918d/ce55ed75-3d20-4bd3-84d2-d62dbd0d02de/6fcf384b-60b0-45a5-8dc1-cf23d8e5c23c"
@@
 		(dnp no)
 		(fields_autoplaced yes)
-		(property "Reference" "R1101"
+		(property "Reference" "R402"
 			(at 148.59 85.09 0)
 			(effects
@@
 		)
 		(instances
+			(project "TEST_PCB"
+				(path "/29496ace-b476-4f24-a65f-9da1dd70122c/59fca87d-eab6-4325-93c7-8130e49f891e/6fcf384b-60b0-45a5-8dc1-cf23d8e5c23c"
+					(reference "R402")
+					(unit 1)
+				)
+			)
 			(project "EPS_CORE"
 				(path "/43e5e7c8-e7e0-4528-9a3e-b1557849918d/ce55ed75-3d20-4bd3-84d2-d62dbd0d02de/6fcf384b-60b0-45a5-8dc1-cf23d8e5c23c"
@@
 		(on_board yes)
 		(dnp no)
-		(property "Reference" "#PWR0324"
+		(property "Reference" "#PWR0168"
 			(at 189.23 128.27 0)
 			(effects
@@
 		)
 		(instances
+			(project "TEST_PCB"
+				(path "/29496ace-b476-4f24-a65f-9da1dd70122c/59fca87d-eab6-4325-93c7-8130e49f891e/6fcf384b-60b0-45a5-8dc1-cf23d8e5c23c"
+					(reference "#PWR0168")
+					(unit 1)
+				)
+			)
 			(project "EPS_CORE"
 				(path "/43e5e7c8-e7e0-4528-9a3e-b1557849918d/ce55ed75-3d20-4bd3-84d2-d62dbd0d02de/6fcf384b-60b0-45a5-8dc1-cf23d8e5c23c"
@@
 		(dnp no)
 		(fields_autoplaced yes)
-		(property "Reference" "R1103"
+		(property "Reference" "R404"
 			(at 173.99 85.09 0)
 			(effects
@@
 		)
 		(instances
+			(project "TEST_PCB"
+				(path "/29496ace-b476-4f24-a65f-9da1dd70122c/59fca87d-eab6-4325-93c7-8130e49f891e/6fcf384b-60b0-45a5-8dc1-cf23d8e5c23c"
+					(reference "R404")
+					(unit 1)
+				)
+			)
 			(project "EPS_CORE"
 				(path "/43e5e7c8-e7e0-4528-9a3e-b1557849918d/ce55ed75-3d20-4bd3-84d2-d62dbd0d02de/6fcf384b-60b0-45a5-8dc1-cf23d8e5c23c"
@@
 		(on_board yes)
 		(dnp no)
-		(property "Reference" "#PWR0327"
+		(property "Reference" "#PWR0171"
 			(at 110.49 109.22 0)
 			(effects
@@
 		)
 		(instances
+			(project "TEST_PCB"
+				(path "/29496ace-b476-4f24-a65f-9da1dd70122c/59fca87d-eab6-4325-93c7-8130e49f891e/6fcf384b-60b0-45a5-8dc1-cf23d8e5c23c"
+					(reference "#PWR0171")
+					(unit 1)
+				)
+			)
 			(project "EPS_CORE"
 				(path "/43e5e7c8-e7e0-4528-9a3e-b1557849918d/ce55ed75-3d20-4bd3-84d2-d62dbd0d02de/6fcf384b-60b0-45a5-8dc1-cf23d8e5c23c"
@@
 		(dnp no)
 		(fields_autoplaced yes)
-		(property "Reference" "R1106"
+		(property "Reference" "R401"
 			(at 139.7 114.2999 0)
 			(effects
@@
 		)
 		(instances
+			(project "TEST_PCB"
+				(path "/29496ace-b476-4f24-a65f-9da1dd70122c/59fca87d-eab6-4325-93c7-8130e49f891e/6fcf384b-60b0-45a5-8dc1-cf23d8e5c23c"
+					(reference "R401")
+					(unit 1)
+				)
+			)
 			(project "EPS_CORE"
 				(path "/43e5e7c8-e7e0-4528-9a3e-b1557849918d/ce55ed75-3d20-4bd3-84d2-d62dbd0d02de/6fcf384b-60b0-45a5-8dc1-cf23d8e5c23c"
@@
 		(dnp no)
 		(fields_autoplaced yes)
-		(property "Reference" "U1101"
+		(property "Reference" "U401"
 			(at 190.1541 86.36 0)
 			(effects
@@
 		)
 		(instances
+			(project "TEST_PCB"
+				(path "/29496ace-b476-4f24-a65f-9da1dd70122c/59fca87d-eab6-4325-93c7-8130e49f891e/6fcf384b-60b0-45a5-8dc1-cf23d8e5c23c"
+					(reference "U401")
+					(unit 1)
+				)
+			)
 			(project "EPS_CORE"
 				(path "/43e5e7c8-e7e0-4528-9a3e-b1557849918d/ce55ed75-3d20-4bd3-84d2-d62dbd0d02de/6fcf384b-60b0-45a5-8dc1-cf23d8e5c23c"
@@
 		(on_board yes)
 		(dnp no)
-		(property "Reference" "#PWR0325"
+		(property "Reference" "#PWR0169"
 			(at 176.53 128.27 0)
 			(effects
@@
 		)
 		(instances
+			(project "TEST_PCB"
+				(path "/29496ace-b476-4f24-a65f-9da1dd70122c/59fca87d-eab6-4325-93c7-8130e49f891e/6fcf384b-60b0-45a5-8dc1-cf23d8e5c23c"
+					(reference "#PWR0169")
+					(unit 1)
+				)
+			)
 			(project "EPS_CORE"
 				(path "/43e5e7c8-e7e0-4528-9a3e-b1557849918d/ce55ed75-3d20-4bd3-84d2-d62dbd0d02de/6fcf384b-60b0-45a5-8dc1-cf23d8e5c23c"
@@
 		(on_board yes)
 		(dnp no)
-		(property "Reference" "R1105"
+		(property "Reference" "R406"
 			(at 208.28 107.9499 0)
 			(effects
@@
 		)
 		(instances
+			(project "TEST_PCB"
+				(path "/29496ace-b476-4f24-a65f-9da1dd70122c/59fca87d-eab6-4325-93c7-8130e49f891e/6fcf384b-60b0-45a5-8dc1-cf23d8e5c23c"
+					(reference "R406")
+					(unit 1)
+				)
+			)
 			(project "EPS_CORE"
 				(path "/43e5e7c8-e7e0-4528-9a3e-b1557849918d/ce55ed75-3d20-4bd3-84d2-d62dbd0d02de/6fcf384b-60b0-45a5-8dc1-cf23d8e5c23c"
@@
 		(on_board yes)
 		(dnp no)
-		(property "Reference" "#PWR0326"
+		(property "Reference" "#PWR0170"
 			(at 139.7 90.17 0)
 			(effects
@@
 		)
 		(instances
+			(project "TEST_PCB"
+				(path "/29496ace-b476-4f24-a65f-9da1dd70122c/59fca87d-eab6-4325-93c7-8130e49f891e/6fcf384b-60b0-45a5-8dc1-cf23d8e5c23c"
+					(reference "#PWR0170")
+					(unit 1)
+				)
+			)
 			(project "EPS_CORE"
 				(path "/43e5e7c8-e7e0-4528-9a3e-b1557849918d/ce55ed75-3d20-4bd3-84d2-d62dbd0d02de/6fcf384b-60b0-45a5-8dc1-cf23d8e5c23c"
@@
 		(dnp yes)
 		(fields_autoplaced yes)
-		(property "Reference" "JP1102"
+		(property "Reference" "JP402"
 			(at 130.81 100.33 0)
 			(effects
@@
 		)
 		(instances
+			(project "TEST_PCB"
+				(path "/29496ace-b476-4f24-a65f-9da1dd70122c/59fca87d-eab6-4325-93c7-8130e49f891e/6fcf384b-60b0-45a5-8dc1-cf23d8e5c23c"
+					(reference "JP402")
+					(unit 1)
+				)
+			)
 			(project "EPS_CORE"
 				(path "/43e5e7c8-e7e0-4528-9a3e-b1557849918d/ce55ed75-3d20-4bd3-84d2-d62dbd0d02de/6fcf384b-60b0-45a5-8dc1-cf23d8e5c23c"

Commit message: nearly finnished CORE pcb
Parts:
- renumbered C401 to C1101, JP401 to JP1101, JP402 to JP1102, R402 to R1101, R403 to R1102, R404 to R1103, R405 to R1104, R406 to R1105, R401 to R1106, U401 to U1101
Connections:
- net A_P renamed A_N
- net B_N renamed B_P
Changed lines of the file:
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@@
 		)
 	)
-	(hierarchical_label "A_P"
+	(hierarchical_label "A_N"
 		(shape bidirectional)
 		(at 219.71 96.52 0)
@@
 		)
 	)
-	(hierarchical_label "B_N"
+	(hierarchical_label "B_P"
 		(shape bidirectional)
 		(at 219.71 101.6 0)
@@
 		(on_board yes)
 		(dnp no)
-		(property "Reference" "R405"
+		(property "Reference" "R1104"
 			(at 208.28 97.7899 0)
 			(effects
@@
 		(on_board yes)
 		(dnp no)
-		(property "Reference" "R403"
+		(property "Reference" "R1102"
 			(at 163.83 85.725 0)
 			(effects
@@
 		(dnp yes)
 		(fields_autoplaced yes)
-		(property "Reference" "JP401"
+		(property "Reference" "JP1101"
 			(at 121.92 91.44 90)
 			(effects
@@
 		(on_board yes)
 		(dnp no)
-		(property "Reference" "#PWR0172"
+		(property "Reference" "#PWR0328"
 			(at 142.24 125.73 0)
 			(effects
@@
 		(dnp no)
 		(fields_autoplaced yes)
-		(property "Reference" "C401"
+		(property "Reference" "C1101"
 			(at 137.16 80.0035 0)
 			(effects
@@
 		(dnp no)
 		(fields_autoplaced yes)
-		(property "Reference" "R402"
+		(property "Reference" "R1101"
 			(at 148.59 85.09 0)
 			(effects
@@
 		(on_board yes)
 		(dnp no)
-		(property "Reference" "#PWR0168"
+		(property "Reference" "#PWR0324"
 			(at 189.23 128.27 0)
 			(effects
@@
 		(dnp no)
 		(fields_autoplaced yes)
-		(property "Reference" "R404"
+		(property "Reference" "R1103"
 			(at 173.99 85.09 0)
 			(effects
@@
 		(on_board yes)
 		(dnp no)
-		(property "Reference" "#PWR0171"
+		(property "Reference" "#PWR0327"
 			(at 110.49 109.22 0)
 			(effects
@@
 		(dnp no)
 		(fields_autoplaced yes)
-		(property "Reference" "R401"
+		(property "Reference" "R1106"
 			(at 139.7 114.2999 0)
 			(effects
@@
 		(dnp no)
 		(fields_autoplaced yes)
-		(property "Reference" "U401"
+		(property "Reference" "U1101"
 			(at 190.1541 86.36 0)
 			(effects
@@
 		(on_board yes)
 		(dnp no)
-		(property "Reference" "#PWR0169"
+		(property "Reference" "#PWR0325"
 			(at 176.53 128.27 0)
 			(effects
@@
 		(on_board yes)
 		(dnp no)
-		(property "Reference" "R406"
+		(property "Reference" "R1105"
 			(at 208.28 107.9499 0)
 			(effects
@@
 		(on_board yes)
 		(dnp no)
-		(property "Reference" "#PWR0170"
+		(property "Reference" "#PWR0326"
 			(at 139.7 90.17 0)
 			(effects
@@
 		(dnp yes)
 		(fields_autoplaced yes)
-		(property "Reference" "JP402"
+		(property "Reference" "JP1102"
 			(at 130.81 100.33 0)
 			(effects
