File: EPS_PC104.kicad_sch (KiCad schematic)
At the start: 2 parts

Commit message: progress on PCBs
Parts:
- renumbered H1701 to H1903, H1702 to H1904
Changed lines of the file:
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@@
 		(on_board yes)
 		(dnp no)
-		(property "Reference" "#PWR?"
+		(property "Reference" "#PWR01911"
 			(at 200.66 134.62 0)
 			(effects
@@
 		(on_board yes)
 		(dnp no)
-		(property "Reference" "#PWR?"
+		(property "Reference" "#PWR01910"
 			(at 172.72 134.62 0)
 			(effects
@@
 		(dnp no)
 		(fields_autoplaced yes)
-		(property "Reference" "H?"
+		(property "Reference" "H1903"
 			(at 134.62 64.77 0)
 			(effects
@@
 		(on_board yes)
 		(dnp no)
-		(property "Reference" "#PWR?"
+		(property "Reference" "#PWR01909"
 			(at 148.59 134.62 0)
 			(effects
@@
 		(dnp no)
 		(fields_autoplaced yes)
-		(property "Reference" "#PWR?"
+		(property "Reference" "#PWR01907"
 			(at 29.21 49.53 0)
 			(effects
@@
 		(dnp no)
 		(fields_autoplaced yes)
-		(property "Reference" "H?"
+		(property "Reference" "H1904"
 			(at 186.69 64.77 0)
 			(effects
@@
 		(on_board yes)
 		(dnp no)
-		(property "Reference" "#PWR?"
+		(property "Reference" "#PWR01908"
 			(at 120.65 134.62 0)
 			(effects
