File: EPS_CORE/EPS_CORE.kicad_pcb (KiCad board)
At the start: 6 copper layers, 90 x 95.8 mm, 304 parts, among them IC1401 TPS259802ONRGER, IC1402 TPS259802ONRGER, IC1601 TPS259802ONRGER, IC1602 TPS259802ONRGER, IC301 TPS259802ONRGER, IC302 TPS259802ONRGER, IC601 TPS259802ONRGER, IC602 TPS259802ONRGER, IC801 TPS259802ONRGER, IC802 TPS259802ONRGER, J102 BATT_PACK, J104 BATT_PACK, J106 OUT, J901 Conn_01x02_Pin, J902 JTAG, J903 JTAG, Q1001 NVTFWS4D9N04XMTAG, Q1002 NVTFWS4D9N04XMTAG, Q1003 BSS138L, Q201 NVTFWS4D9N04XMTAG, Q202 NVTFWS4D9N04XMTAG, SW101 Deploy, U1001 TPS62933, U1002 LM74700, U1003 TPS62933, U1004 LM74700, U101 LP38690SDX-3.3/NOPB, U1101 THVD1424, U1701 TMCS1101A2UQDT, U1801 TMCS1101A2UQDT, U201 LM74700, U202 LM74700, U401 TMCS1101A2UQDT, U901 LP38690SDX-3.3/NOPB, U902 MSP430FR5969IRGZR, U903 ADG1607xCP, U904 MSP430FR5969IRGZR, U905 TCAN4551RGYRQ1, U906 ADG1607xCP, Y901 Crystal, Y902 Crystal

Commit message: nearly finnished CORE pcb
Parts:
- removed C920, C931: 10u, Capacitor_SMD:C_1206_3216Metric_Pad1.33x1.80mm_HandSolder
- removed J901: Conn_01x02_Pin, Connector_PinHeader_2.54mm:PinHeader_1x02_P2.54mm_Vertical
- added FID103: Fiducial, Fiducial:Fiducial_1mm_Mask2mm, B.Cu at (51.2, 54.1)
- added FID104: Fiducial, Fiducial:Fiducial_1mm_Mask2mm, B.Cu at (125.0, 114.8)
- added J101: CAN, Connector_Molex:Molex_PicoBlade_53261-0471_1x04-1MP_P1.25mm_Horizontal, F.Cu at (126.7, 60.0)
- added J103: RS-485, Connector_Molex:Molex_PicoBlade_53261-0471_1x04-1MP_P1.25mm_Horizontal, F.Cu at (126.7, 72.7)
- added R1205: 0, Resistor_SMD:R_0603_1608Metric_Pad0.98x0.95mm_HandSolder, F.Cu at (88.2, 60.1)
- added R1207: 0, Resistor_SMD:R_0603_1608Metric_Pad0.98x0.95mm_HandSolder, F.Cu at (89.8, 60.1)
- added R1209: 0, Resistor_SMD:R_0603_1608Metric_Pad0.98x0.95mm_HandSolder, F.Cu at (86.6, 60.1)
- added R1210: 0, Resistor_SMD:R_0603_1608Metric_Pad0.98x0.95mm_HandSolder, F.Cu at (85.0, 60.1)
- C1601, C1602, C1603, C1604, C1605, C1606, C1607, C1608, C1801, C1802, C1803, C201, C202, C203, C204, C205, C206, C301, C302, C303, C304, C305, C306, C307, C308, C401, C402, C403, C601, C602, C603, C604, C605, C606, C607, C608, C801, C802, C803, C804, C805, C806, C807, C808, IC1601, IC1602, IC301, IC302, IC601, IC602, IC801, IC802, Q201, Q202, R103, R104, R1501, R1502, R1601, R1602, R1603, R1604, R1605, R1606, R1607, R1608, R1609, R1610, R1611, R1612, R201, R301, R302, R303, R304, R305, R306, R307, R308, R309, R310, R311, R312, R501, R502, R601, R602, R603, R604, R605, R606, R607, R608, R609, R610, R611, R612, R701, R702, R801, R802, R803, R804, R805, R806, R807, R808, R809, R810, R811, R812, R913, TP1601, TP1602, TP301, TP302, TP601, TP602, TP801, TP802, U1801, U201, U202, U401: moved to B.Cu
- J102, J104: footprint Connector_Harwin:Harwin_Gecko-G125-FVX1605L0X_2x08_P1.25mm_Vertical -> Outlines:G125-MH11605L1P; moved to B.Cu
- J106: footprint Connector_Harwin:Harwin_Gecko-G125-MVX1005L1X_2x05_P1.25mm_Vertical -> Outlines:G125-MH11605L1P; moved to B.Cu
- R101: footprint Resistor_SMD:R_0603_1608Metric_Pad0.98x0.95mm_HandSolder -> Resistor_SMD:R_1210_3225Metric_Pad1.30x2.65mm_HandSolder
- R102: footprint Resistor_SMD:R_0603_1608Metric_Pad0.98x0.95mm_HandSolder -> Resistor_SMD:R_1210_3225Metric_Pad1.30x2.65mm_HandSolder; moved to B.Cu
- moved R104 184.4 mm to (83.6, 104.0), turned to 180 degrees
- moved R103 180.1 mm to (80.1, 104.0), turned to 180 degrees
- moved TP302 178.7 mm to (80.0, 93.9)
- moved IC302 177.8 mm to (80.3, 99.0)
- moved C308 172.3 mm to (86.4, 97.8), turned to 90 degrees
- moved C304 171.4 mm to (86.4, 111.0), turned to 90 degrees
- moved TP301 169.9 mm to (79.8, 107.6)
- moved C307 169.7 mm to (84.7, 97.8), turned to 90 degrees
- moved C303 168.8 mm to (84.7, 111.0), turned to 90 degrees
- moved R312 168.7 mm to (85.1, 93.3), turned to 90 degrees
- moved IC301 168.6 mm to (80.3, 112.4)
- moved C305 167.6 mm to (73.6, 97.7), turned to 90 degrees
- moved R310 164.6 mm to (83.5, 93.3), turned to 90 degrees
- moved R306 164.0 mm to (84.9, 107.0), turned to 90 degrees
- moved C306 163.5 mm to (76.6, 93.3), turned to 90 degrees
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Connections:
- C1701 pad 1: +5V -> +3V3
- C1801 pad 1: +5V -> +3V3
- C401 pad 1: +5V -> +3V3
- H101 pad 10: /Ch_AL_5 -> /Ch_V_3
- H101 pad 11: /AMEAS_5 -> /AMEAS_SOL_6
- H101 pad 12: /Ch_AL_3 -> /Ch_V_2
- H101 pad 13: /AMEAS_6 -> /AMEAS_SOL_4
- H101 pad 14: /Ch_AL_6 -> /Ch_V_1
- H101 pad 15: /AMEAS_7 -> /AMEAS_SOL_2
- H101 pad 16: /Ch_AL_7 -> /Ch_AL_6
- H101 pad 17: /AMEAS_8 -> /AMEAS_SOL_1
- H101 pad 18: /Ch_AL_8 -> /Ch_AL_5
- H101 pad 21: /Ch_EN_11 -> /MPPT_~{EN}
- H101 pad 22: /Ch_V_8 -> GND
- H101 pad 23: /Ch_EN_41 -> /Ch_EN_22
- H101 pad 24: /Ch_V_7 -> GND
- H101 pad 25: /Ch_EN_12 -> /Ch_EN_32
- H101 pad 26: /SOL_EN_6 -> /Ch_EN_7x
- H101 pad 27: /Ch_EN_42 -> /Ch_EN_12
- H101 pad 28: /SOL_EN_5 -> /Ch_EN_8x
- H101 pad 29: /Ch_EN_21 -> /Ch_EN_11
- H101 pad 30: /SOL_EN_4 -> /Ch_EN_21
- H101 pad 31: /Ch_EN_51 -> /Ch_EN_41
- H101 pad 32: /SOL_EN_3 -> /SOL_STAT_2
- H101 pad 33: /Ch_EN_22 -> /SOL_EN_1
- H101 pad 35: /Ch_EN_52 -> /SOL_EN_3
- H101 pad 36: /SOL_EN_1 -> /SOL_EN_4
- H101 pad 4: /Ch_AL_1 -> /Ch_V_6
- H101 pad 5: /AMEAS_2 -> /AMEAS_3
- H101 pad 6: /Ch_AL_4 -> /Ch_V_5
- H101 pad 7: /AMEAS_3 -> /AMEAS_5
- H101 pad 8: /Ch_AL_2 -> /Ch_V_4
- H101 pad 9: /AMEAS_4 -> /AMEAS_7
- H102 pad 10: /VMEAS_SOL_4 -> /AMEAS_8
- H102 pad 11: /Ch_V_2 -> /Ch_AL_7
- H102 pad 12: /VMEAS_SOL_5 -> /AMEAS_SOL_5
- H102 pad 13: /Ch_V_1 -> /Ch_AL_8
- H102 pad 14: /VMEAS_SOL_6 -> /AMEAS_SOL_3
- H102 pad 18: /AMEAS_SOL_1 -> /VMEAS_SOL_1
- H102 pad 19: GND -> /Ch_V_7
- H102 pad 20: /AMEAS_SOL_2 -> /VMEAS_SOL_2
- H102 pad 21: GND -> /Ch_V_8
- H102 pad 22: /AMEAS_SOL_3 -> /VMEAS_SOL_3
- H102 pad 24: /AMEAS_SOL_4 -> /VMEAS_SOL_4
- H102 pad 26: /AMEAS_SOL_5 -> /VMEAS_SOL_5
- H102 pad 27: /MPPT_~{EN} -> /Ch_EN_42
- H102 pad 28: /AMEAS_SOL_6 -> /VMEAS_SOL_6
- H102 pad 3: /Ch_V_6 -> /Ch_AL_1
- H102 pad 31: /Ch_EN_61 -> /Ch_EN_62
- H102 pad 32: /SOL_STAT_2 -> /Ch_EN_52
- H102 pad 33: /Ch_EN_32 -> /Ch_EN_61
- H102 pad 34: /SOL_STAT_1 -> /Ch_EN_51
- H102 pad 35: /Ch_EN_62 -> /SOL_EN_5
- H102 pad 37: /Ch_EN_7x -> /SOL_STAT_1
- H102 pad 38: /Ch_EN_8x -> /SOL_EN_6
- H102 pad 5: /Ch_V_5 -> /Ch_AL_2
- H102 pad 6: /VMEAS_SOL_2 -> /AMEAS_4
- H102 pad 7: /Ch_V_4 -> /Ch_AL_3
- H102 pad 8: /VMEAS_SOL_3 -> /AMEAS_6
- H102 pad 9: /Ch_V_3 -> /Ch_AL_4
- H1201 pad 25: +5V -> Net-(H1201-Pin_25)
- H1201 pad 26: +5V -> Net-(H1201-Pin_26)
- H1201 pad 27: +3V3 -> Net-(H1201-Pin_27)
- H1201 pad 28: +3V3 -> Net-(H1201-Pin_28)
- J102 pad 13: /AMEAS_9 -> GND
- J102 pad 15: SCL -> GND
- J102 pad 16: /HEAT_BATT_1 -> /BATT_BOOT
- J102 pad 4: GND -> /TMEAS_BATT_1
- J102 pad 5: /ALERT -> /BATT_ALERT_1
- J102 pad 6: GND -> SCL
- J102 pad 8: +3V3 -> /HEAT_BATT_1
- J104 pad 13: /TMEAS_BATT_2 -> GND
- J104 pad 15: SCL -> GND
- J104 pad 16: /HEAT_BATT_2 -> /BATT_BOOT
- J104 pad 4: GND -> /TMEAS_BATT_2
- J104 pad 5: /ALERT -> /BATT_ALERT_2
- J104 pad 6: GND -> SCL
- J104 pad 8: +3V3 -> /HEAT_BATT_2
- J902 pad MP: (no net) -> SHIELD
- J903 pad MP: (no net) -> SHIELD
- R1104 pad 1: /RS_Rx_N -> /RS_Rx_P
- R1104 pad 2: /RS_Rx_P -> /RS_Rx_N
- U1101 pad 11: /RS_Rx_N -> /RS_Rx_P
- U1101 pad 12: /RS_Rx_P -> /RS_Rx_N
- U1701 pad 8: +5V -> +3V3
- U1801 pad 8: +5V -> +3V3
- U401 pad 8: +5V -> +3V3
- U902 pad 3: /MCU/ADC_3 -> /MCU/ADC_4
- U902 pad 33: /MCU/AMUX_0 -> /MCU/AMUX_EN
- U902 pad 34: /MCU/AMUX_1 -> /MCU/AMUX_0
- U902 pad 35: /MCU/AMUX_2 -> /MCU/AMUX_1
- U902 pad 39: /MCU/AMUX_EN -> /MCU/AMUX_2
- U902 pad 6: /BATT_ALERT_1 -> /BATT_ALERT_2
- U902 pad 7: /BATT_ALERT_2 -> /BATT_ALERT_1
- U902 pad 9: /MCU/ADC_4 -> /MCU/ADC_3
- U903 pad 7: /AMEAS_10 -> /TMEAS_BATT_2
- U903 pad 8: /AMEAS_9 -> /TMEAS_BATT_1
- U904 pad 38: /MCU/BATT_BOOT -> /BATT_BOOT
- U906 pad 19: /AMEAS_2 -> /VMEAS_SOL_1
- U906 pad 7: /TMEAS_BATT_2 -> /AMEAS_10
Routing:
- net GND: track 190.1 -> 740.2 mm, vias 126 -> 776
- net +3V3: track 6.32 -> 152.4 mm, vias 0 -> 8
- net /BATT_BOOT: track 0.00 -> 107.3 mm, vias 0 -> 3
- net /Ch_AL_9: track 8.53 -> 108.4 mm
- net /BUS: track 0.00 -> 98.2 mm, vias 0 -> 22
- net SDA: track 56.7 -> 142.1 mm, vias 2 -> 3
- net /Ch_EN_92: track 9.68 -> 95.1 mm, vias 1 -> 2
- net /AMEAS_BUS: track 3.29 -> 85.5 mm, vias 1 -> 3
- net /MCU/CAN_~{INT}: track 5.27 -> 83.2 mm
- net SCL: track 55.7 -> 133.0 mm, vias 0 -> 2
- net /Ch_AL_10: track 2.30 -> 77.3 mm, vias 1 -> 4
- net /Switch_Deploy_BUS/EN: track 0.00 -> 74.4 mm, vias 0 -> 3
- net /MCU/CAN_~{WKRQ}: track 5.20 -> 78.2 mm, vias 2 -> 3
- net /Ch_EN_102: track 2.32 -> 71.3 mm, vias 1 -> 2
- net /AMEAS_10: track 2.22 -> 68.1 mm, vias 1 -> 3
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- added copper zone on B.Cu, net /AMEAS_10/VIN
- added copper zone on B.Cu, net /AMEAS_10/VOUT
- added copper zone on B.Cu, net /AMEAS_9/VOUT
- added copper zone on B.Cu, net /AMEAS_BUS/VIN
- added copper zone on B.Cu, net /BATT_PACK_1
- added copper zone on B.Cu, net /BATT_PACK_2
- added copper zone on B.Cu, net /BUS
- added copper zone on In2.Cu, net /BUS
- added copper zone on B.Cu, net /Channel_10
- added copper zone on B.Cu, net /Channel_9
- added copper zone on B.Cu, net /Switch_Deploy_BUS/Switch_Element/VOUT1
- added copper zone on B.Cu, net /Switch_Deploy_BUS/Switch_Element/VOUT2
