File: EPS_OUTPUT_CHANNELS/EPS_OUTPUT_CHANNELS.kicad_pcb (KiCad board)
At the start: 6 copper layers, 90 x 95.8 mm, 370 parts, among them IC1001 TPS259802ONRGER, IC1002 TPS259802ONRGER, IC1201 TPS259802ONRGER, IC1202 TPS259802ONRGER, IC1401 TPS259802ONRGER, IC1402 TPS259802ONRGER, IC801 TPS259802ONRGER, IC802 TPS259802ONRGER, J102 Channel, J103 Channel, J104 Channel, J107 Channel, Q1301 NVTFWS4D9N04XMTAG, Q1302 NVTFWS4D9N04XMTAG, Q201 NVTFWS4D9N04XMTAG, Q202 NVTFWS4D9N04XMTAG, Q203 BSS138L, Q301 NVTFWS4D9N04XMTAG, Q302 NVTFWS4D9N04XMTAG, Q303 BSS138L, Q401 NVTFWS4D9N04XMTAG, Q402 NVTFWS4D9N04XMTAG, Q403 BSS138L, Q501 NVTFWS4D9N04XMTAG, Q502 NVTFWS4D9N04XMTAG, Q503 BSS138L, U1301 LM74700, U1302 LM74700, U1501 TMCS1101A2UQDT, U1601 TMCS1101A2UQDT, U1701 TMCS1101A2UQDT, U1801 TMCS1101A2UQDT, U201 TPS62933, U202 LM74700, U203 TPS62933, U204 LM74700, U301 TPS62933, U302 LM74700, U303 TPS62933, U304 LM74700, U401 TPS62933, U402 LM74700, U403 TPS62933, U404 LM74700, U501 TPS62933, U502 LM74700, U503 TPS62933, U504 LM74700

Commit message: progress on PCBs
Parts:
- removed H101, H102: PC104, Connector_PinSocket_2.54mm:PinSocket_2x26_P2.54mm_Vertical
- added C601: 1u, Capacitor_SMD:C_0603_1608Metric_Pad1.08x0.95mm_HandSolder, F.Cu at (203.6, 117.0)
- added C602: SELECT, Capacitor_SMD:C_0603_1608Metric_Pad1.08x0.95mm_HandSolder, F.Cu at (203.6, 119.6)
- added C603: SELECT, Capacitor_SMD:C_0603_1608Metric_Pad1.08x0.95mm_HandSolder, F.Cu at (203.6, 122.1)
- added C604: 1u, Capacitor_SMD:C_0603_1608Metric_Pad1.08x0.95mm_HandSolder, F.Cu at (203.6, 124.6)
- added C605: 1u, Capacitor_SMD:C_0603_1608Metric_Pad1.08x0.95mm_HandSolder, F.Cu at (223.5, 117.0)
- added C606: SELECT, Capacitor_SMD:C_0603_1608Metric_Pad1.08x0.95mm_HandSolder, F.Cu at (223.5, 119.5)
- added C607: SELECT, Capacitor_SMD:C_0603_1608Metric_Pad1.08x0.95mm_HandSolder, F.Cu at (223.5, 122.0)
- added C608: 1u, Capacitor_SMD:C_0603_1608Metric_Pad1.08x0.95mm_HandSolder, F.Cu at (223.5, 124.5)
- added H1903: PC104, Connector_PinSocket_2.54mm:PinSocket_2x26_P2.54mm_Vertical, F.Cu at (102.9, 118.6)
- added H1904: PC104, Connector_PinSocket_2.54mm:PinSocket_2x26_P2.54mm_Vertical, F.Cu at (102.9, 123.8)
- added IC601: TPS259830ONRGER, Outlines:TPS259830ONRGER, F.Cu at (217.1, 103.0)
- added IC602: TPS259830ONRGER, Outlines:TPS259830ONRGER, F.Cu at (217.2, 89.6)
- added Q601: NVTFWS4D9N04XMTAG, Outlines:NVTFS5116PLTWG, F.Cu at (198.8, 129.7)
- added Q602: NVTFWS4D9N04XMTAG, Outlines:NVTFS5116PLTWG, F.Cu at (223.7, 128.7)
- added R601: 0, Resistor_SMD:R_1210_3225Metric_Pad1.30x2.65mm_HandSolder, F.Cu at (211.3, 128.7)
- added R602: SELECT, Resistor_SMD:R_0603_1608Metric_Pad0.98x0.95mm_HandSolder, F.Cu at (207.9, 117.0)
- added R603: SELECT, Resistor_SMD:R_0603_1608Metric_Pad0.98x0.95mm_HandSolder, F.Cu at (207.9, 119.6)
- added R604: 10, Resistor_SMD:R_0603_1608Metric_Pad0.98x0.95mm_HandSolder, F.Cu at (207.9, 122.1)
- added R605: SELECT, Resistor_SMD:R_0603_1608Metric_Pad0.98x0.95mm_HandSolder, F.Cu at (207.9, 124.6)
- added R606: SELECT, Resistor_SMD:R_0603_1608Metric_Pad0.98x0.95mm_HandSolder, F.Cu at (212.3, 117.0)
- added R607: SELECT, Resistor_SMD:R_0603_1608Metric_Pad0.98x0.95mm_HandSolder, F.Cu at (212.3, 119.6)
- added R608: SELECT, Resistor_SMD:R_0603_1608Metric_Pad0.98x0.95mm_HandSolder, F.Cu at (212.3, 122.1)
- added R609: SELECT, Resistor_SMD:R_0603_1608Metric_Pad0.98x0.95mm_HandSolder, F.Cu at (212.3, 124.6)
- added R610: 0, Resistor_SMD:R_1210_3225Metric_Pad1.30x2.65mm_HandSolder, F.Cu at (230.9, 127.9)
- added R611: SELECT, Resistor_SMD:R_0603_1608Metric_Pad0.98x0.95mm_HandSolder, F.Cu at (227.9, 117.0)
- added R612: SELECT, Resistor_SMD:R_0603_1608Metric_Pad0.98x0.95mm_HandSolder, F.Cu at (227.9, 119.5)
- added R613: 10, Resistor_SMD:R_0603_1608Metric_Pad0.98x0.95mm_HandSolder, F.Cu at (227.9, 122.0)
- added R614: SELECT, Resistor_SMD:R_0603_1608Metric_Pad0.98x0.95mm_HandSolder, F.Cu at (227.9, 124.5)
- added R615: SELECT, Resistor_SMD:R_0603_1608Metric_Pad0.98x0.95mm_HandSolder, F.Cu at (232.2, 117.0)
- added R616: SELECT, Resistor_SMD:R_0603_1608Metric_Pad0.98x0.95mm_HandSolder, F.Cu at (232.2, 119.5)
- added R617: SELECT, Resistor_SMD:R_0603_1608Metric_Pad0.98x0.95mm_HandSolder, F.Cu at (232.2, 122.0)
- added R618: SELECT, Resistor_SMD:R_0603_1608Metric_Pad0.98x0.95mm_HandSolder, F.Cu at (232.2, 124.5)
- C1301, C1302, C1303, C1304, C1305, C1306, C1401, C1402, C1403, C1404, C1405, C1406, C1407, C1408, C1801, C1802, C1803, C501, C502, C503, C504, C505, C506, C507, C508, C510, C511, C512, C513, C514, C515, C516, C517, C518, C519, C521, C522, C523, C524, IC1401, IC1402, L501, L502, Q1301, Q1302, Q501, Q502, Q503, R124, R126, R130, R1301, R1401, R1402, R1403, R1404, R1405, R1406, R1407, R1408, R1409, R1410, R1411, R1412, R150, R151, R501, R502, R503, R504, R505, R506, R507, R508, R509, R510, TP1401, TP1402, U1301, U1302, U1801, U501, U502, U503, U504: moved to F.Cu
- J102: moved to B.Cu
- moved TP1401 192.9 mm to (318.4, 110.0), turned to 180 degrees
- moved TP1402 190.6 mm to (318.3, 97.1), turned to 180 degrees
- moved C1401 186.9 mm to (325.3, 113.7), turned to 90 degrees
- moved IC1401 186.9 mm to (318.5, 115.3), turned to 180 degrees
- moved C1405 186.2 mm to (325.1, 100.8), turned to 90 degrees
- moved IC1402 185.8 mm to (318.6, 102.1), turned to 180 degrees
- moved C1402 183.2 mm to (321.8, 109.7), turned to 90 degrees
- moved R1401 182.6 mm to (323.6, 113.7), turned to -90 degrees
- moved R1402 182.0 mm to (323.4, 109.7), turned to -90 degrees
- moved C1403 177.2 mm to (314.2, 113.9), turned to 90 degrees
- moved C1406 176.6 mm to (321.8, 96.6), turned to -90 degrees
- moved C1404 176.2 mm to (312.6, 113.9), turned to 90 degrees
- moved R1407 176.0 mm to (323.4, 100.8), turned to -90 degrees
- moved R1405 173.5 mm to (320.1, 109.7), turned to 90 degrees
- moved C1407 170.1 mm to (314.3, 100.7), turned to 90 degrees
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Connections:
- C1302 pad 1: /AMEAS_7/VIN -> /Switch_CH_7/VOUT
- C1305 pad 1: /AMEAS_7/VIN -> /Switch_CH_7/VOUT
- C1401 pad 1: /DCDC_7/VOUT -> /Switch_CH_7/VIN1
- C1405 pad 1: /DCDC_7/VOUT -> /Switch_CH_7/VIN2
- IC1401 pad 1: /DCDC_7/VOUT -> /Switch_CH_7/VIN1
- IC1401 pad 13: /Ch_AL_7/8 -> /Switch_CH_7/PG
- IC1401 pad 16: /DCDC_7/VOUT -> /Switch_CH_7/VIN1
- IC1401 pad 2: /DCDC_7/VOUT -> /Switch_CH_7/VIN1
- IC1401 pad 25: /DCDC_7/VOUT -> /Switch_CH_7/VIN1
- IC1401 pad 3: /DCDC_7/VOUT -> /Switch_CH_7/VIN1
- IC1401 pad 6: /Ch_EN_7x/8 -> /Switch_CH_7/EN
- IC1402 pad 1: /DCDC_7/VOUT -> /Switch_CH_7/VIN2
- IC1402 pad 13: /Ch_AL_7/8 -> /Switch_CH_7/PG
- IC1402 pad 16: /DCDC_7/VOUT -> /Switch_CH_7/VIN2
- IC1402 pad 2: /DCDC_7/VOUT -> /Switch_CH_7/VIN2
- IC1402 pad 25: /DCDC_7/VOUT -> /Switch_CH_7/VIN2
- IC1402 pad 3: /DCDC_7/VOUT -> /Switch_CH_7/VIN2
- IC1402 pad 6: /Ch_EN_7x/8 -> /Switch_CH_7/EN
- Q1301 pad 1: /AMEAS_7/VIN -> /Switch_CH_7/VOUT
- Q1302 pad 1: /AMEAS_7/VIN -> /Switch_CH_7/VOUT
- R1301 pad 2: /Ch_EN_7x/8 -> /Switch_CH_7/EN
- R1401 pad 1: /Ch_EN_7x/8 -> /Switch_CH_7/EN
- R1401 pad 2: /DCDC_7/VOUT -> /Switch_CH_7/VIN1
- R1402 pad 2: /Ch_EN_7x/8 -> /Switch_CH_7/EN
- R1407 pad 1: /Ch_EN_7x/8 -> /Switch_CH_7/EN
- R1407 pad 2: /DCDC_7/VOUT -> /Switch_CH_7/VIN2
- R1408 pad 2: /Ch_EN_7x/8 -> /Switch_CH_7/EN
- U1301 pad 4: /AMEAS_7/VIN -> /Switch_CH_7/VOUT
- U1302 pad 4: /AMEAS_7/VIN -> /Switch_CH_7/VOUT
Routing:
- net VBUS: track 19.5 -> 104.5 mm, vias 1 -> 22
- net /Ch_AL_2/5: track 1.70 -> 76.2 mm, vias 0 -> 4
- net /AMEAS_2/5: track 1.60 -> 62.9 mm, vias 0 -> 3
- net /Ch_V_6: track 0.00 -> 53.8 mm, vias 0 -> 1
- net /AMEAS_3/6: track 1.60 -> 46.1 mm, vias 0 -> 3
- net /Ch_EN_12/4: track 1.60 -> 45.8 mm, vias 0 -> 1
- net /Ch_EN_11/4: track 1.60 -> 43.7 mm, vias 0 -> 1
- net /Ch_V_3: track 0.00 -> 37.4 mm, vias 0 -> 1
- net Net-(Q203-D): track 0.00 -> 37.1 mm
- net Net-(Q303-D): track 0.00 -> 36.7 mm
- net /AMEAS_7/8: track 1.60 -> 37.1 mm, vias 0 -> 1
- net /Ch_EN_21/5: track 1.60 -> 36.5 mm, vias 0 -> 2
- net GND: track 71.9 -> 106.6 mm, vias 19 -> 499
- net /Ch_V_1/4: track 1.60 -> 34.6 mm, vias 0 -> 1
- net /Ch_EN_32/6: track 8.99 -> 41.5 mm, vias 0 -> 2
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- added copper zone on F.Cu, net /AMEAS_1/VIN
- added copper zone on F.Cu, net /AMEAS_1/VOUT
- added copper zone on B.Cu, net /AMEAS_2/VIN
- added copper zone on B.Cu, net /AMEAS_2/VOUT
- added copper zone on F.Cu, net /Channel_1
- added copper zone on B.Cu, net /Channel_2
- added copper zone on F.Cu, net /DCDC_1/VOUT
- added copper zone on B.Cu, net /DCDC_2/VOUT
- added copper zone on F.Cu, net Net-(Q201-S)
- added copper zone on F.Cu, net Net-(Q202-S)
- added copper zone on B.Cu, net Net-(Q301-S)
- added copper zone on B.Cu, net Net-(Q302-S)
- added copper zone on F.Cu, net Net-(U201-SW)
- added copper zone on F.Cu, net Net-(U203-SW)
- added copper zone on B.Cu, net Net-(U301-SW)
- added copper zone on B.Cu, net Net-(U303-SW)
- added copper zone on B.Cu, net VBUS
