File: EPS_PV_INPUT/EPS_PV_INPUT.kicad_pcb (KiCad board)
At the start: 6 copper layers, 90 x 95.8 mm, 488 parts, among them IC1301 TPS259802ONRGER, IC1302 TPS259802ONRGER, IC1701 TPS259802ONRGER, IC1702 TPS259802ONRGER, IC2101 TPS259802ONRGER, IC2102 TPS259802ONRGER, IC2501 TPS259802ONRGER, IC2502 TPS259802ONRGER, IC501 TPS259802ONRGER, IC502 TPS259802ONRGER, IC901 TPS259802ONRGER, IC902 TPS259802ONRGER, J102 PV, J103 PV, J104 PV, J105 PV, J106 PV, J108 PV, Q1001 NVTFWS4D9N04XMTAG, Q1002 NVTFWS4D9N04XMTAG, Q1003 BSS138L, Q1201 NVTFWS4D9N04XMTAG, Q1202 NVTFWS4D9N04XMTAG, Q1401 NVTFWS4D9N04XMTAG, Q1402 NVTFWS4D9N04XMTAG, Q1403 BSS138L, Q1601 NVTFWS4D9N04XMTAG, Q1602 NVTFWS4D9N04XMTAG, Q1801 NVTFWS4D9N04XMTAG, Q1802 NVTFWS4D9N04XMTAG, Q1803 BSS138L, Q2001 NVTFWS4D9N04XMTAG, Q2002 NVTFWS4D9N04XMTAG, Q201 NVTFWS4D9N04XMTAG, Q202 NVTFWS4D9N04XMTAG, Q203 BSS138L, Q2201 NVTFWS4D9N04XMTAG, Q2202 NVTFWS4D9N04XMTAG, Q2203 BSS138L, Q2401 NVTFWS4D9N04XMTAG, Q2402 NVTFWS4D9N04XMTAG, Q401 NVTFWS4D9N04XMTAG, Q402 NVTFWS4D9N04XMTAG, Q601 NVTFWS4D9N04XMTAG, Q602 NVTFWS4D9N04XMTAG, Q603 BSS138L, Q801 NVTFWS4D9N04XMTAG, Q802 NVTFWS4D9N04XMTAG, U1001 BQ24650, U1101 TMCS1101A2UQDT, U1201 LM74700, U1202 LM74700, U1401 BQ24650, U1501 TMCS1101A2UQDT, U1601 LM74700, U1602 LM74700, U1801 BQ24650, U1901 TMCS1101A2UQDT, U2001 LM74700, U2002 LM74700, U201 BQ24650, U2201 BQ24650, U2301 TMCS1101A2UQDT, U2401 LM74700, U2402 LM74700, U301 TMCS1101A2UQDT, U401 LM74700, U402 LM74700, U601 BQ24650, U701 TMCS1101A2UQDT, U801 LM74700, U802 LM74700

Commit message: progress on PCBs
Parts:
- moved C402 0.23 mm to (164.1, 64.2)
Routing:
- net Net-(D201-K): track 0.07 -> 8.89 mm
- net +3V3: track 0.00 -> 2.49 mm
- net /BUS: track 8.27 -> 6.34 mm
- net Net-(Q201-G): track 17.1 -> 17.6 mm
- net GND: vias 64 -> 69
- added copper zone on F.Cu, net GND
